File: audio_back_plane_35_rca.kicad_pcb (KiCad board)
At the start: 4 copper layers, 100 x 75 mm, 91 parts, among them IC1 TMUX4053DYYR, IC2 SN74LVC245ARGYR, IC3 TMUX4052BQBR, IC4 TMUX4053BQBR, J1 header, Q1 IRLML6344TRPBF, Q2 IRLML6344TRPBF, SW1 RotaryEncoder_Switch_MP, SW2 TL1105WF160Q - 3.15mm actuator, SW3 TL1105WF160Q - 3.15mm actuator, SW4 TL1105WF160Q - 3.15mm actuator, SW5 TL1105WF160Q - 3.15mm actuator, SW6 TL1105WF160Q - 3.15mm actuator, U1 Teensy 4.1 - DEVKIT, U2 ESP32-DevKitC - DEVKIT, U4 EN11-HSM1AF15

Commit message: update
Parts:
- removed HPTRS3: 3.5MM JACK, project_fp:35RAPC3BH3
- removed the HPTRS4 at (155.0, 66.6)
- removed IC1: TMUX4053DYYR, SamacSys_Parts:SOP50P326X110-16N
- removed IC3: TMUX4052BQBR, SamacSys_Parts:TMUX4052BQBR
- removed IC4: TMUX4053BQBR, SamacSys_Parts:TMUX4053BQBR
- removed Q1, Q2: IRLML6344TRPBF, SamacSys_Parts:SOT95P237X112-3N
- removed R21, R23, R24, R25: 6.8k, project_fp:R_0805_2012Metric_Pad1.20x1.40mm_HandSolder
- removed S1: PEC12R-2220F-S0024, project_fp:XDCR_PEC12R-2220F-S0024
- removed USBB1: USB B Device (Optional) - B1HSxx, project_fp:USB_B_OST_USB-B1HSxx_Horizontal
- removed USB_IN1, USB_THRU1: header, project_fp:USB_IN1
- added J3: Conn_Coaxial_x2, project_fp:PJRAS2X1_NOT-VERIFIED, F.Cu at (88.5, 75.6)
- added J4: Conn_01x08, Connector_PinHeader_2.54mm:PinHeader_1x08_P2.54mm_Vertical, F.Cu at (89.1, 85.0)
- added J5: NMJ6HFD2-AU, Connector_Audio:Jack_6.35mm_Neutrik_NMJ6HFD2-AU_Horizontal, F.Cu at (93.2, 124.2)
- added J6: Conn_Coaxial_x2, project_fp:PJRAS2X1_NOT-VERIFIED, F.Cu at (118.5, 75.6)
- Brd1, D10, D11, D12, D13, D14, D15, D16, D17, D18, D19, D2, D20, D21, D22, D3, D5, D6, D7, D8, D9, SW1, SW2, SW3, SW4, SW5, SW6, U4: moved to F.Cu
- D1, D4: footprint project_fp:PinHeader_1x04_P1.00mm_Vertical_WS2812_LED_mod -> project_fp:PinHeader_1x04_P2.54mm_Vertical
- board_outline2: footprint project_fp:audio_project_board_outline_100x75 -> project_fp:audio_project_board_outline_125x75
- moved SW6 579.7 mm to (555.5, 253.0), turned to 0 degrees
- moved D22 511.3 mm to (593.0, 266.6), turned to 0 degrees
- moved D20 508.2 mm to (593.0, 260.4), turned to 0 degrees
- moved D18 506.4 mm to (589.9, 266.6), turned to 0 degrees
- moved D21 506.3 mm to (593.0, 263.5), turned to 0 degrees
- moved D19 503.4 mm to (593.0, 257.4), turned to 0 degrees
- moved D16 503.4 mm to (589.9, 260.4), turned to 0 degrees
- moved D17 501.5 mm to (589.9, 263.5), turned to 0 degrees
- moved D15 498.7 mm to (589.9, 257.4), turned to 0 degrees
- moved D8 497.3 mm to (583.8, 260.4), turned to 0 degrees
- moved D7 486.2 mm to (583.8, 257.4), turned to 0 degrees
- moved U4 485.7 mm to (605.0, 244.4)
- moved MIC2 460.0 mm to (541.0, 245.7)
- moved C2 460.0 mm to (540.3, 241.6)
- moved SW2 459.4 mm to (555.5, 222.6), turned to 0 degrees
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Connections:
- HPTRS1 pad 2: Net-(IC1-D1) -> unconnected-(HPTRS1-Pad2)
- HPTRS1 pad 5: Net-(IC4-SEL3) -> unconnected-(HPTRS1-Pad5)
- HPTRS2 pad 1: GND -> unconnected-(HPTRS2-Pad1)
- HPTRS2 pad 2: Net-(IC1-D3) -> unconnected-(HPTRS2-Pad2)
- HPTRS2 pad 5: Net-(IC1-D2) -> unconnected-(HPTRS2-Pad5)
- HPTRS4 pad 3: Net-(board_outline1-IN1M) -> unconnected-(HPTRS4-Pad3)
- TDM1 pad 1: (no net) -> 35_TX8_RESET
- TDM1 pad 10: (no net) -> GND
- TDM1 pad 11: (no net) -> Net-(TDM1-BCLK)
- TDM1 pad 12: (no net) -> GND
- TDM1 pad 13: (no net) -> Net-(TDM1-LRCK)
- TDM1 pad 14: (no net) -> GND
- TDM1 pad 15: (no net) -> SDA_C
- TDM1 pad 16: (no net) -> GND
- TDM1 pad 17: (no net) -> SCL_C
- TDM1 pad 18: (no net) -> GND
- TDM1 pad 19: (no net) -> Net-(TDM1-MCLK)
- TDM1 pad 2: (no net) -> 34_RX8_RESET2
- TDM1 pad 20: (no net) -> GND
- TDM1 pad 3: (no net) -> 5V
- TDM1 pad 4: (no net) -> SYSTEM_EN
- TDM1 pad 5: (no net) -> 12V
- TDM1 pad 6: (no net) -> GND
- TDM1 pad 7: (no net) -> Net-(TDM1-DSP_DATA_IN)
- TDM1 pad 8: (no net) -> GND
- TDM1 pad 9: (no net) -> Net-(TDM1-DSP_DATA_OUT)
- board_outline1 pad 21: Net-(IC1-S2B) -> unconnected-(board_outline1-OUTP-Pad21)
- board_outline1 pad 23: Net-(IC1-S1A) -> unconnected-(board_outline1-OUT1M-Pad23)
- board_outline1 pad 25: Net-(IC1-S1B) -> unconnected-(board_outline1-OUT2P-Pad25)
- board_outline1 pad 27: Net-(IC1-S3B) -> unconnected-(board_outline1-OUT2M-Pad27)
- board_outline1 pad 29: Net-(board_outline1-IN1P) -> unconnected-(board_outline1-IN1P-Pad29)
- board_outline1 pad 31: Net-(board_outline1-IN1M) -> unconnected-(board_outline1-IN1M-Pad31)
Routing:
- net 5V: track 133.1 -> 0.00 mm, vias 3 -> 0
- net 3.3V: track 129.1 -> 0.00 mm, vias 4 -> 0
- net /SWITCH: track 98.7 -> 0.00 mm, vias 1 -> 0
- net /OUTPUTA: track 81.0 -> 0.00 mm, vias 1 -> 0
- net 35_TX8_RESET: track 79.9 -> 0.00 mm, vias 2 -> 0
- net Net-(MIC1-DATA): track 78.1 -> 0.00 mm, vias 2 -> 0
- net Net-(MIC1-BCLK-PDMCLK): track 72.8 -> 0.00 mm
- net /OUTPUTB: track 63.6 -> 0.00 mm, vias 2 -> 0
- net 2_OUT2: track 62.8 -> 0.00 mm
- net ESP32_IO12_SPI_MISO: track 57.0 -> 0.00 mm
- net ESP32_IO13_SPI_MOSI: track 56.7 -> 0.00 mm
- net 5_IN2: track 49.1 -> 0.00 mm
- net ESP32_IO0: track 47.5 -> 0.00 mm
- net Net-(IC1-S2B): track 47.3 -> 0.00 mm
- net HOST_5V: track 43.1 -> 0.00 mm
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Other:
- board size 100 x 75 mm -> 125 x 75 mm
- board text removed: "< VOL >"
- board text removed: "BT WIFI"
- board text removed: "IN1"
- board text removed: "IN2"
- board text removed: "MIC"
- board text removed: "NEXT"
- board text removed: "OUT1"
- board text removed: "PLAY REC"
- board text removed: "PLAY/PAUSE"
- board text removed: "PREV"
- board text removed: "SD"
- board text removed: "SELECT MODE"
- board text removed: "USB"

Commit message: update
Parts:
- removed Brd1: SSD1306, project_fp:Adafruit_SSD1306_I2C_ONLY
- removed C1, C3, C4, C6: 0.1uF, project_fp:C_0805_2012Metric_Pad1.15x1.40mm_HandSolder
- removed D10, D11, D12, D13, D14, D15, D16, D17, D18, D19, D2, D20, D21, D22, D3, D5, D6, D7, D8, D9: SK6812, project_fp:LED_SK6812_EC15_1.5x1.5mm
- removed HPTRS2: 3.5MM JACK, project_fp:35RAPC3BH3
- removed IC2: SN74LVC245ARGYR, SamacSys_Parts:SN74LVC541ARGYR
- removed J1: header, project_fp:PinHeader_1x02_P2.54mm_Vertical_W_CUT
- removed J5: NMJ6HFD2-AU, Connector_Audio:Jack_6.35mm_Neutrik_NMJ6HFD2-AU_Horizontal
- removed R11, R7: 470 ohm, project_fp:R_0805_2012Metric_Pad1.20x1.40mm_HandSolder
- removed R13, R14, R15: 10k, project_fp:R_0805_2012Metric_Pad1.20x1.40mm_HandSolder
- removed SW1: RotaryEncoder_Switch_MP, project_fp:RotaryEncoder_Alps_EC11E_Vertical_H20mm
- removed SW2, SW3, SW4: TL1105WF160Q - 3.15mm actuator, project_fp:Tactile_Switch_4.54.5MM
- removed TDM1 (x2): header, project_fp:T-DSP_Expansion_Header_2x10_ALT_GND
- removed U4: EN11-HSM1AF15, project_fp:EN11-HSM_TTE
- added 1/4-PHONE1: NMJ6HFD2-AU, project_fp:Jack_6.35mm_Neutrik_NMJ6HCD3_Horizontal, F.Cu at (85.7, 143.5)
- added C11: 0.1uF, project_fp:C_0805_2012Metric_Pad1.15x1.40mm_HandSolder, F.Cu at (157.0, 64.5)
- added C16: 0.1uF, project_fp:C_0805_2012Metric_Pad1.15x1.40mm_HandSolder, F.Cu at (86.4, 61.2)
- added C17: 0.1uF, project_fp:C_0805_2012Metric_Pad1.15x1.40mm_HandSolder, F.Cu at (86.2, 66.6)
- added C18: 0.1uF, project_fp:C_0805_2012Metric_Pad1.15x1.40mm_HandSolder, F.Cu at (86.5, 71.5)
- added C19: 0.1uF, project_fp:C_0805_2012Metric_Pad1.15x1.40mm_HandSolder, F.Cu at (86.5, 76.7)
- added C20: 0.1uF, project_fp:C_0805_2012Metric_Pad1.15x1.40mm_HandSolder, F.Cu at (86.5, 81.8)
- added C21: 0.1uF, project_fp:C_0805_2012Metric_Pad1.15x1.40mm_HandSolder, F.Cu at (121.0, 154.5)
- added C22: 0.1uF, project_fp:C_0805_2012Metric_Pad1.15x1.40mm_HandSolder, F.Cu at (123.0, 162.3)
- added C31: 0.1uF, project_fp:C_0805_2012Metric_Pad1.15x1.40mm_HandSolder, F.Cu at (146.9, 153.6)
- added C32: 0.1uF, project_fp:C_0805_2012Metric_Pad1.15x1.40mm_HandSolder, F.Cu at (146.9, 156.5)
- added C8: 0.1uF, project_fp:C_0805_2012Metric_Pad1.15x1.40mm_HandSolder, F.Cu at (141.4, 65.2)
- added D23: Diode - 1N4148, project_fp:D_SOD-123, F.Cu at (141.7, 72.4)
- added H1: MountingHole_Pad, MountingHole:MountingHole_3.2mm_M3_DIN965_Pad, F.Cu at (81.0, 88.5)
- added H2: MountingHole_Pad, MountingHole:MountingHole_3.2mm_M3_DIN965_Pad, F.Cu at (178.5, 88.0)
- added H3: MountingHole_Pad, MountingHole:MountingHole_3.2mm_M3_DIN965_Pad, F.Cu at (81.0, 114.5)
- added H6: MountingHole_Pad, MountingHole:MountingHole_3.2mm_M3_DIN965_Pad, F.Cu at (179.0, 130.0)
- added IN1: jumper, project_fp:SolderJumper-3_P_12_BRIDGED, F.Cu at (91.0, 61.2)
- added MIDI_IN_1: 3.5mm TRS - 35RAPC3BH3, project_fp:35RAPC3BH3, F.Cu at (169.4, 43.9)
- added MIDI_IO1: header, project_fp:MIDI_IO1, F.Cu at (177.2, 64.2)
- added OUTA1: jumper, project_fp:SolderJumper-3_P_23_BRIDGED, F.Cu at (91.2, 66.5)
- added OUTB1: jumper, project_fp:SolderJumper-3_P_23_BRIDGED, F.Cu at (92.0, 81.9)
- added OUTC1: jumper, project_fp:SolderJumper-3_P_23_BRIDGED, F.Cu at (91.7, 76.2)
- added OUTD1: jumper, project_fp:SolderJumper-3_P_23_BRIDGED, F.Cu at (91.3, 71.3)
- added PWR1: LED_1206, Diode_SMD:D_1210_3225Metric_Pad1.42x2.65mm_HandSolder, F.Cu at (127.8, 68.4)
- added R21: 0ohm, project_fp:R_0805_2012Metric_Pad1.20x1.40mm_HandSolder, F.Cu at (161.8, 64.3)
- added R22: 220 ohm, project_fp:R_0805_2012Metric_Pad1.20x1.40mm_HandSolder, F.Cu at (161.8, 67.3)
- added R23: 1.5k, project_fp:R_0805_2012Metric_Pad1.20x1.40mm_HandSolder, F.Cu at (157.0, 67.4)
- added R24: 220 ohm, project_fp:R_0805_2012Metric_Pad1.20x1.40mm_HandSolder, F.Cu at (141.4, 68.1)
- added R25: 0ohm, project_fp:R_0805_2012Metric_Pad1.20x1.40mm_HandSolder, F.Cu at (157.0, 70.4)
- added R26: 47 ohm, project_fp:R_0805_2012Metric_Pad1.20x1.40mm_HandSolder, F.Cu at (161.8, 70.2)
- added R27: 220 ohm, project_fp:R_0805_2012Metric_Pad1.20x1.40mm_HandSolder, F.Cu at (161.8, 73.2)
- added R28: 220 ohm, project_fp:R_0805_2012Metric_Pad1.20x1.40mm_HandSolder, F.Cu at (161.8, 76.1)
- added R29: 47 ohm, project_fp:R_0805_2012Metric_Pad1.20x1.40mm_HandSolder, F.Cu at (161.8, 79.1)
- added R30: 0 ohm, project_fp:R_0805_2012Metric_Pad1.20x1.40mm_HandSolder, F.Cu at (79.3, 105.8)
- added R31: 0 ohm, project_fp:R_0805_2012Metric_Pad1.20x1.40mm_HandSolder, F.Cu at (79.2, 95.9)
- added R35: 49.9 ohm, project_fp:R_0805_2012Metric_Pad1.20x1.40mm_HandSolder, F.Cu at (79.9, 61.4)
- added RLED1: led, project_fp:R_0805_2012Metric_Pad1.20x1.40mm_HandSolder, F.Cu at (132.8, 68.5)
- added SW7: SW_SPST, project_fp:SW_Tactile_SPST_Angled_PTS645Vx39-2LFS, F.Cu at (137.0, 156.5)
- added SW8: SW_SPST, project_fp:SW_Tactile_SPST_Angled_PTS645Vx39-2LFS, F.Cu at (137.0, 165.9)
- added TDM3: header, project_fp:T-DSP_Expansion_Header_2x10_ALT_GND, F.Cu at (67.8, 102.7)
- added TDM4: header, project_fp:T-DSP_Expansion_Header_2x10_ALT_GND, F.Cu at (68.1, 65.9)
- added U10: SN74LVC1T45DBV, Package_TO_SOT_SMD:SOT-23-6, F.Cu at (83.0, 66.5)
- added U11: SN74LVC1T45DBV, Package_TO_SOT_SMD:SOT-23-6, F.Cu at (83.3, 71.4)
- added U12: SN74LVC1T45DBV, Package_TO_SOT_SMD:SOT-23-6, F.Cu at (83.5, 76.6)
- added U13: SN74LVC1T45DBV, Package_TO_SOT_SMD:SOT-23-6, F.Cu at (83.4, 81.7)
- added U14: Single Buffer - 74LVC1G125GV,125 - SOT-23-5/SC-74A/SOT-753, Package_TO_SOT_SMD:SOT-23-5, F.Cu at (83.3, 96.0)
- added U5: Optoisolators - H11L1SM - 6-SMD, Gull Wing, project_fp:IC_H11L1SM, F.Cu at (149.0, 69.5)
- added U6: Dual Buffer - 74HCT2G17GW,125 - SOT-363_SC-70-6, project_fp:SOT-363_SC-70-6, F.Cu at (157.1, 74.0)
- added U7: Single Buffer - 74LVC1G125GV,125 - SOT-23-5/SC-74A/SOT-753, Package_TO_SOT_SMD:SOT-23-5, F.Cu at (83.1, 100.7)
- added U8: Single Buffer - 74LVC1G125GV,125 - SOT-23-5/SC-74A/SOT-753, Package_TO_SOT_SMD:SOT-23-5, F.Cu at (83.1, 105.8)
- added U9: SN74LVC1T45DBV, Package_TO_SOT_SMD:SOT-23-6, F.Cu at (83.3, 61.2)
- G1: moved to B.Cu
- J3: value Conn_Coaxial_x2 -> RCA-IN
- J6: value Conn_Coaxial_x2 -> RCA-OUT
- MIC1: value SPH0655LM4H-1 -> SPH0645LM4H-B
- R16: value 0 ohm -> 49.9 ohm
- R20: value 49.9 ohm -> 0 ohm
- SW5: value TL1105WF160Q - 3.15mm actuator -> SW_SPST; footprint project_fp:Tactile_Switch_4.54.5MM -> project_fp:SW_Tactile_SPST_Angled_PTS645Vx39-2LFS
- SW6: footprint project_fp:Tactile_Switch_4.54.5MM -> project_fp:SW_Tactile_SPST_Angled_PTS645Vx39-2LFS
- U1: footprint project_fp:Teensy41_mod2 -> project_fp:Teensy41_mod
- board_outline2: footprint project_fp:audio_project_board_outline_125x75 -> project_fp:audio_project_board_outline_100x120
- moved C2 463.5 mm to (105.8, 80.3), turned to 90 degrees
- moved MIC2 461.7 mm to (109.8, 80.7)
- moved SW5 453.6 mm to (111.2, 153.7)
- moved SW6 453.6 mm to (111.2, 161.3)
- moved MIC1 436.8 mm to (109.8, 115.7), turned to 180 degrees
- moved board_outline2 122.7 mm to (183.1, 143.8), turned to 90 degrees
- moved C5 61.1 mm to (105.6, 115.6), turned to 90 degrees
- moved C7 53.1 mm to (136.2, 54.6), turned to -90 degrees
- moved R9 52.6 mm to (137.8, 109.5)
- moved G1 48.0 mm to (151.7, 50.5), turned to 0 degrees
- moved R16 31.6 mm to (79.9, 66.2), turned to -90 degrees
- moved CC1 29.2 mm to (139.2, 54.6)
- moved CC2 29.2 mm to (142.2, 54.6)
- moved USBA1 28.4 mm to (153.8, 43.7)
- moved board_outline1 27.5 mm to (96.8, 82.7), turned to -90 degrees
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Connections:
- HPTRS1 pad 2: unconnected-(HPTRS1-Pad2) -> Net-(1/4-PHONE1-PadRN)
- HPTRS1 pad 3: unconnected-(HPTRS1-Pad3) -> Net-(J6-IN2)
- HPTRS1 pad 4: unconnected-(HPTRS1-Pad4) -> Net-(J6-IN1)
- HPTRS1 pad 5: unconnected-(HPTRS1-Pad5) -> Net-(1/4-PHONE1-PadTN)
- HPTRS4 pad 2: Net-(board_outline1-IN2M) -> Net-(board_outline1-IN1P)
- HPTRS4 pad 3: unconnected-(HPTRS4-Pad3) -> Net-(J3-IN2)
- J3 pad 1: unconnected-(J3-IN1-Pad1) -> IN2_JACK_DETECT
- J3 pad 2: unconnected-(J3-IN2-Pad2) -> Net-(J3-IN2)
- J6 pad 1: unconnected-(J6-IN1-Pad1) -> Net-(J6-IN1)
- J6 pad 2: unconnected-(J6-IN2-Pad2) -> Net-(J6-IN2)
- R16 pad 1: Net-(TDM1-DSP_DATA_IN) -> 7_OUT1A+
- R17 pad 1: Net-(TDM1-DSP_DATA_OUT) -> 6_OUT1D+
- R18 pad 1: Net-(TDM1-BCLK) -> 9_OUT1C+
- R18 pad 2: BCLK1+ -> Net-(U12-B)
- R19 pad 1: Net-(TDM1-LRCK) -> 32_OUT1B+
- R19 pad 2: LRCK1+ -> Net-(U13-B)
- R20 pad 1: Net-(TDM1-MCLK) -> MCLK1+
- R20 pad 2: MCLK1+ -> Net-(U7-Y)
- SW5 pad 1: T_BUTTON1 -> 53_T_PROG
- SW5 pad 2: unconnected-(SW5-B-Pad2) -> GND
- SW6 pad 1: T_BUTTON2 -> 54_ON_OFF
- SW6 pad 2: unconnected-(SW6-B-Pad2) -> GND
- board_outline1 pad 21: unconnected-(board_outline1-OUTP-Pad21) -> Net-(board_outline1-OUTP)
- board_outline1 pad 25: unconnected-(board_outline1-OUT2P-Pad25) -> Net-(board_outline1-OUT2P)
- board_outline1 pad 29: unconnected-(board_outline1-IN1P-Pad29) -> Net-(board_outline1-IN1P)
- board_outline1 pad 35: Net-(board_outline1-IN2M) -> unconnected-(board_outline1-IN2M-Pad35)
Other:
- board size 125 x 75 mm -> 120 x 100 mm

Commit message: update
Parts:
- removed R12: 2.2k ohm - 2200 ohm, project_fp:R_0805_2012Metric_Pad1.20x1.40mm_HandSolder
- added C1: 0.1uF, project_fp:C_0805_2012Metric_Pad1.15x1.40mm_HandSolder, F.Cu at (196.5, 78.1)
- added C3: 0.1uF, project_fp:C_0805_2012Metric_Pad1.15x1.40mm_HandSolder, F.Cu at (196.5, 81.1)
- added ESP_I1: header, project_fp:ESP_I2C_0_PinHeader_2x02_P2.54mm_Vertical, F.Cu at (177.7, 121.7)
- added ESP_R_ENC1: header, project_fp:ESP_R_ENC0_PinHeader_1x05_P2.54mm_Vertical, F.Cu at (180.5, 107.9)
- added GPI1: header, project_fp:GPI1_PinHeader_1x04_P2.54mm_Vertical, F.Cu at (180.7, 94.8)
- added ILI1: ILI9341+XPT2046, project_fp:ILI9341_PinHeader_1x14_P2.54mm_Vertical, F.Cu at (177.5, 85.0)
- added ILI_VCC1: jumper, project_fp:SolderJumper-3_P1.3mm_Bridged2Bar12_Pad1.0x1.5mm_NumberLabels, F.Cu at (186.7, 102.7)
- added R11: 470 ohm, project_fp:R_0805_2012Metric_Pad1.20x1.40mm_HandSolder, F.Cu at (270.6, 79.0)
- added R46: 2.2k ohm - 2200 ohm, project_fp:R_0805_2012Metric_Pad1.20x1.40mm_HandSolder, F.Cu at (246.0, 103.5)
- added R47: 2.2k ohm - 2200 ohm, project_fp:R_0805_2012Metric_Pad1.20x1.40mm_HandSolder, F.Cu at (246.0, 106.5)
- added R48: 2.2k ohm - 2200 ohm, project_fp:R_0805_2012Metric_Pad1.20x1.40mm_HandSolder, F.Cu at (246.0, 109.4)
- added R59: 2.2k ohm - 2200 ohm, project_fp:R_0805_2012Metric_Pad1.20x1.40mm_HandSolder, F.Cu at (246.0, 112.3)
- added R60: 2.2k ohm - 2200 ohm, project_fp:R_0805_2012Metric_Pad1.20x1.40mm_HandSolder, F.Cu at (246.0, 115.3)
- added R7: 470 ohm, project_fp:R_0805_2012Metric_Pad1.20x1.40mm_HandSolder, F.Cu at (196.5, 84.0)
- moved SW5 170.0 mm to (266.4, 84.2), turned to -90 degrees
- moved SW6 168.8 mm to (266.3, 94.7), turned to -90 degrees
- moved C21 153.9 mm to (258.1, 84.5), turned to -90 degrees
- moved C22 150.7 mm to (258.1, 95.5), turned to -90 degrees
- moved SW7 138.5 mm to (265.9, 105.7), turned to -90 degrees
- moved SW8 138.2 mm to (266.4, 117.2), turned to -90 degrees
- moved C31 120.4 mm to (257.6, 106.0), turned to -90 degrees
- moved C32 116.9 mm to (257.3, 117.7), turned to -90 degrees
- moved D4 43.3 mm to (203.0, 78.2)
- moved D1 38.5 mm to (209.5, 78.7)
- moved H2 11.5 mm to (179.0, 76.5)
- moved MIDI_IO1 8.14 mm to (178.7, 56.1)
Connections:
- U2 pad 33: unconnected-(U2-GPIO21-Pad33) -> /ESP32_IO21_SDA
- U2 pad 36: unconnected-(U2-GPIO22-Pad36) -> /ESP32_IO22_SCL
- U2 pad 5: unconnected-(U2-VDET_1/GPIO34/ADC1_CH6-Pad5) -> Net-(GPI1-Pin_2)
- U2 pad 6: unconnected-(U2-VDET_2/GPIO35/ADC1_CH7-Pad6) -> Net-(GPI1-Pin_1)

Commit message: update
Parts:
- removed D4: HEADER, project_fp:PinHeader_1x04_P2.54mm_Vertical
- removed SW5, SW7, SW8: SW_SPST, project_fp:SW_Tactile_SPST_Angled_PTS645Vx39-2LFS
- removed SW6: TL1105WF160Q - 3.15mm actuator, project_fp:SW_Tactile_SPST_Angled_PTS645Vx39-2LFS
- added C26: 0.1uF, project_fp:C_0805_2012Metric_Pad1.15x1.40mm_HandSolder, F.Cu at (87.0, 96.0)
- added C27: 0.1uF, project_fp:C_0805_2012Metric_Pad1.15x1.40mm_HandSolder, F.Cu at (86.5, 100.5)
- added C28: 0.1uF, project_fp:C_0805_2012Metric_Pad1.15x1.40mm_HandSolder, F.Cu at (86.5, 106.0)
- added D2: SK6812, project_fp:LED_4691, F.Cu at (135.9, 142.5)
- added D5: SK6812, project_fp:LED_4691, F.Cu at (130.4, 142.5)
- added R12: 0 ohm, project_fp:R_0805_2012Metric_Pad1.20x1.40mm_HandSolder, F.Cu at (130.4, 140.0)
- added R13: 0 ohm, project_fp:R_0805_2012Metric_Pad1.20x1.40mm_HandSolder, F.Cu at (136.4, 140.0)
- added T_PROG1: header, project_fp:T_PROG1_PinHeader_1x03_P2.54mm_Vertical, F.Cu at (176.5, 74.5)
- added T_PROG2: header, project_fp:E_PROG1_PinHeader_1x03_P2.54mm_Vertical, F.Cu at (180.0, 74.5)
- added U15: Single Buffer - 74LVC1G125GV,125 - SOT-23-5/SC-74A/SOT-753, Package_TO_SOT_SMD:SOT-23-5, F.Cu at (130.4, 137.0)
- added U16: Single Buffer - 74LVC1G125GV,125 - SOT-23-5/SC-74A/SOT-753, Package_TO_SOT_SMD:SOT-23-5, F.Cu at (136.4, 137.0)
- ILI_VCC1: moved to B.Cu
- moved R11 141.2 mm to (131.9, 105.4)
- moved C21 132.5 mm to (129.9, 118.1)
- moved C22 132.5 mm to (129.9, 129.1)
- moved C32 103.6 mm to (154.5, 104.5)
- moved C31 98.3 mm to (159.5, 100.5)
- moved R46 88.1 mm to (158.5, 113.5)
- moved R47 88.1 mm to (158.5, 116.4)
- moved R48 88.1 mm to (158.5, 119.4)
- moved R59 88.1 mm to (158.5, 122.3)
- moved R60 88.1 mm to (158.5, 125.3)
- moved C1 86.5 mm to (130.4, 134.0)
- moved C3 80.1 mm to (136.4, 134.0), turned to 180 degrees
- moved R7 39.5 mm to (158.5, 95.0)
- moved D1 31.7 mm to (179.0, 87.5)
- moved ILI_VCC1 19.2 mm to (167.5, 101.5), turned to 90 degrees
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Connections:
- D1 pad 1: Net-(D1-Pin_1) -> ESP32_LED+
- D1 pad 2: 5V -> TEENSY_LED+
- D1 pad 4: unconnected-(D1-Pin_4-Pad4) -> 5V
- R11 pad 1: Net-(D4-Pin_1) -> TEENSY_LED
- R11 pad 2: TEENSY_LED -> Net-(U1-41_A17)
- R7 pad 1: Net-(D1-Pin_1) -> Net-(U2-*GPIO5)
- U1 pad 33: TEENSY_LED -> Net-(U1-41_A17)
- U2 pad 29: ESP32_LED -> Net-(U2-*GPIO5)

Commit message: update
Parts:
- removed H1, H2, H3, H6: MountingHole_Pad, MountingHole:MountingHole_3.2mm_M3_DIN965_Pad
- removed J3: RCA-IN, project_fp:PJRAS2X1_NOT-VERIFIED
- removed J6: RCA-OUT, project_fp:PJRAS2X1_NOT-VERIFIED
- added J1: PJRAS2X1S01X, project_fp:PJRAS2X1S01X_MOD2, F.Cu at (122.0, 100.0)
- added J2: PJRAS2X1S01X, project_fp:PJRAS2X1S01X_MOD2, F.Cu at (152.0, 100.0)
- D1: footprint project_fp:PinHeader_1x04_P2.54mm_Vertical -> project_fp:LED_GPIO_PinHeader_1x04_P2.54mm_Vertical
- moved board_outline2 93.9 mm to (100.0, 100.0), turned to -90 degrees
- moved PWR1 83.2 mm to (171.4, 122.7)
- moved RLED1 83.2 mm to (176.4, 122.8)
- moved C8 83.2 mm to (185.0, 119.5)
- moved D23 83.2 mm to (185.3, 126.7)
- moved R23 83.2 mm to (200.6, 121.8)
- moved R24 83.2 mm to (185.0, 122.5)
- moved R25 83.2 mm to (200.6, 124.7)
- moved R26 83.2 mm to (205.4, 124.6)
- moved R27 83.2 mm to (205.4, 127.5)
- moved R28 83.2 mm to (205.4, 130.5)
- moved U5 83.2 mm to (192.6, 123.9)
- moved U6 83.2 mm to (200.7, 128.3)
- moved C11 83.2 mm to (200.6, 118.8)
- moved R21 83.2 mm to (205.4, 118.7)
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- renumbered T_PROG2 to ESP_PROG1
Routing:
- removed copper zone on B.Cu, net GND
- removed copper zone on F.Cu, net GND
- removed copper zone on In1.Cu, net GND
- removed copper zone on In2.Cu, net GND

Commit message: update
Parts:
- moved U1 30.8 mm to (168.0, 200.0), turned to 180 degrees
- moved TDM3 11.7 mm to (102.0, 167.0), turned to 90 degrees
- moved TDM4 9.47 mm to (102.0, 130.0), turned to 90 degrees
- moved board_outline1 6.50 mm to (131.0, 133.0)
- moved HPTRS4 4.19 mm to (150.0, 200.0), turned to 180 degrees
- moved J4 3.68 mm to (129.0, 150.4)
- moved HPTRS1 2.76 mm to (138.0, 200.0), turned to 180 degrees
- moved D5 2.62 mm to (165.0, 200.0), turned to 180 degrees
- moved C1 2.31 mm to (165.0, 190.0)
- moved C3 2.31 mm to (171.0, 190.0)
- moved R12 2.31 mm to (165.0, 196.0)
- moved R13 2.31 mm to (171.0, 196.0)
- moved U15 2.31 mm to (165.0, 193.0)
- moved U16 2.31 mm to (171.0, 193.0)
- moved D2 2.19 mm to (171.0, 200.0), turned to 180 degrees
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