File: audio_back_plane_35_rca.kicad_pcb (KiCad board)
At the start: 4 copper layers, 100 x 61 mm, 69 parts, among them IC1 TMUX4053DYYR, IC2 SN74LVC245ARGYR, J3 header, J4 header, SW1 RotaryEncoder_Switch_MP, SW2 TL1105WF160Q - 3.15mm actuator, SW3 TL1105WF160Q - 3.15mm actuator, SW4 TL1105WF160Q - 3.15mm actuator, SW5 TL1105WF160Q - 3.15mm actuator, SW6 TL1105WF160Q - 3.15mm actuator, U1 Teensy 4.1 - DEVKIT, U2 ESP32-DevKitC - DEVKIT

Commit message: update
Parts:
- removed J4: header, project_fp:PinHeader_1x02_P2.54mm_Vertical_W_CUT
- removed the R17 at (17.0, 155.4)
- removed the R19 at (21.8, 149.5)
- removed the TDM1 at (-5.33, 138.6)
- removed TDM2: header, project_fp:T-DSP_Expansion_Header_2x10_ALT_GND
- added Brd1: SSD1306, project_fp:Adafruit_SSD1306_I2C_ONLY, B.Cu at (148.5, 83.9)
- added CC1: 5.1k, project_fp:R_0805_2012Metric_Pad1.20x1.40mm_HandSolder, F.Cu at (236.9, 98.9)
- added CC2: 5.1k, project_fp:R_0805_2012Metric_Pad1.20x1.40mm_HandSolder, F.Cu at (236.9, 101.8)
- added D13: SK6812, project_fp:LED_SK6812_EC15_1.5x1.5mm, B.Cu at (165.3, 101.5)
- added D14: SK6812, project_fp:LED_SK6812_EC15_1.5x1.5mm, B.Cu at (165.5, 89.0)
- added D15: SK6812, project_fp:LED_SK6812_EC15_1.5x1.5mm, B.Cu at (112.9, 111.8)
- added D16: SK6812, project_fp:LED_SK6812_EC15_1.5x1.5mm, B.Cu at (112.8, 99.8)
- added D17: SK6812, project_fp:LED_SK6812_EC15_1.5x1.5mm, B.Cu at (112.9, 108.8)
- added D18: SK6812, project_fp:LED_SK6812_EC15_1.5x1.5mm, B.Cu at (112.8, 96.8)
- added D19: SK6812, project_fp:LED_SK6812_EC15_1.5x1.5mm, B.Cu at (112.9, 105.7)
- added D20: SK6812, project_fp:LED_SK6812_EC15_1.5x1.5mm, B.Cu at (112.8, 93.7)
- added D21: SK6812, project_fp:LED_SK6812_EC15_1.5x1.5mm, B.Cu at (112.9, 102.7)
- added D22: SK6812, project_fp:LED_SK6812_EC15_1.5x1.5mm, B.Cu at (112.8, 90.7)
- added G2: jumper, project_fp:SolderJumper-2_P1.3mm_Open_TrianglePad1.0x1.5mm, F.Cu at (236.7, 105.1)
- added HPTRS4: 3.5MM JACK, project_fp:35RAPC3BH3, F.Cu at (155.0, 66.6)
- added IC3: TMUX4052BQBR, SamacSys_Parts:TMUX4052BQBR, F.Cu at (95.1, 122.7)
- added IC4: TMUX4053BQBR, SamacSys_Parts:TMUX4053BQBR, F.Cu at (90.1, 122.7)
- added Q1: IRLML6344TRPBF, SamacSys_Parts:SOT95P237X112-3N, F.Cu at (44.9, 123.9)
- added Q2: IRLML6344TRPBF, SamacSys_Parts:SOT95P237X112-3N, F.Cu at (44.9, 119.3)
- added R24: 6.8k, project_fp:R_0805_2012Metric_Pad1.20x1.40mm_HandSolder, F.Cu at (50.1, 122.9)
- added TDM1: header, project_fp:T-DSP_Expansion_Header_2x10_ALT_GND, F.Cu at (89.8, 75.7)
- added TDM1: header, project_fp:T-DSP_Expansion_Header_2x10_ALT_GND, F.Cu at (89.8, 109.7)
- added U4: EN11-HSM1AF15, project_fp:EN11-HSM_TTE, B.Cu at (140.1, 104.0)
- added USBB1: USB B Device (Optional) - B1HSxx, project_fp:USB_B_OST_USB-B1HSxx_Horizontal, F.Cu at (220.8, 88.6)
- added USBC1: USB C Device - USB4085-GF-A, project_fp:GCT_USB4085-GF-A_REVA4, F.Cu at (138.9, 71.3)
- added USB_IN1: header, project_fp:USB_IN1, F.Cu at (239.2, 82.1)
- added USB_THRU1: header, project_fp:USB_IN1, F.Cu at (243.8, 82.1)
- D12: footprint project_fp:LED_SK6812 -> project_fp:LED_SK6812_EC15_1.5x1.5mm; moved to B.Cu
- D9: moved to B.Cu
- R21, R23, R25: value 49.9 ohm -> 6.8k
- board_outline2: footprint project_fp:audio_project_board_outline_60.96x100 -> project_fp:audio_project_board_outline_100x75
- moved C1 328.6 mm to (321.9, 125.7)
- moved C3 328.6 mm to (321.9, 128.7)
- moved D1 328.6 mm to (321.2, 137.6)
- moved R11 328.6 mm to (321.9, 134.6)
- moved R7 328.6 mm to (321.9, 131.6)
- moved D4 328.6 mm to (324.6, 137.6)
- moved SW6 181.4 mm to (-15.3, 151.9)
- moved D9 163.7 mm to (165.3, 107.6), turned to 90 degrees
- moved D12 162.4 mm to (165.5, 92.0), turned to 90 degrees
- moved board_outline2 120.8 mm to (85.4, 141.5), turned to 0 degrees
- moved IC2 120.0 mm to (178.1, 115.5)
- moved S1 94.3 mm to (54.6, 140.7)
- moved SW1 58.3 mm to (200.4, 112.2)
- moved SW3 52.2 mm to (170.3, 120.7), turned to 180 degrees
- moved D11 49.4 mm to (165.3, 104.5), turned to 90 degrees
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- renumbered J3 to J1, R18 to R17, R20 to R18, R22 to R19, R24 to R20
Connections:
- D10 pad 1: unconnected-(D10-VDD-Pad1) -> 5V
- D10 pad 3: unconnected-(D10-GND-Pad3) -> GND
- D10 pad 4: unconnected-(D10-DIN-Pad4) -> Net-(D10-DIN)
- D11 pad 1: unconnected-(D11-VDD-Pad1) -> 5V
- D11 pad 2: unconnected-(D11-DOUT-Pad2) -> Net-(D11-DOUT)
- D11 pad 3: unconnected-(D11-GND-Pad3) -> GND
- D11 pad 4: unconnected-(D11-DIN-Pad4) -> Net-(D11-DIN)
- D12 pad 1: unconnected-(D12-VDD-Pad1) -> 5V
- D12 pad 2: unconnected-(D12-DOUT-Pad2) -> Net-(D12-DOUT)
- D12 pad 3: unconnected-(D12-VSS-Pad3) -> GND
- D12 pad 4: unconnected-(D12-DIN-Pad4) -> Net-(D11-DOUT)
- D3 pad 2: unconnected-(D3-DOUT-Pad2) -> Net-(D3-DOUT)
- D3 pad 3: unconnected-(D3-GND-Pad3) -> GND
- D6 pad 2: unconnected-(D6-DOUT-Pad2) -> Net-(D6-DOUT)
- D7 pad 1: unconnected-(D7-VDD-Pad1) -> 5V
- D7 pad 2: unconnected-(D7-DOUT-Pad2) -> Net-(D7-DOUT)
- D7 pad 3: unconnected-(D7-GND-Pad3) -> GND
- D7 pad 4: unconnected-(D7-DIN-Pad4) -> Net-(D6-DOUT)
- D8 pad 1: unconnected-(D8-VDD-Pad1) -> 5V
- D8 pad 2: unconnected-(D8-DOUT-Pad2) -> Net-(D11-DIN)
- D8 pad 3: unconnected-(D8-GND-Pad3) -> GND
- D8 pad 4: unconnected-(D8-DIN-Pad4) -> Net-(D7-DOUT)
- D9 pad 1: unconnected-(D9-VDD-Pad1) -> 5V
- D9 pad 2: unconnected-(D9-DOUT-Pad2) -> Net-(D10-DIN)
- D9 pad 3: unconnected-(D9-GND-Pad3) -> GND
- D9 pad 4: unconnected-(D9-DIN-Pad4) -> Net-(D3-DOUT)
- HPTRS1 pad 5: Net-(IC1-S2B) -> Net-(IC4-SEL3)
- R21 pad 1: Net-(TDM2-BCLK) -> Net-(Q1-S)
- R21 pad 2: BCLK1+ -> Net-(board_outline1-IN2M)
- R23 pad 1: Net-(TDM2-LRCK) -> Net-(Q1-S)
- R23 pad 2: LRCK1+ -> Net-(board_outline1-IN2P)
- R25 pad 2: MCLK1+ -> Net-(board_outline1-IN1P)
Routing:
- net Net-(U2-ADC2_CH0/GPIO4): track 0.00 -> 23.5 mm, vias 0 -> 1
- net ESP32_LED: track 23.5 -> 0.00 mm, vias 1 -> 0
- net 5V: track 153.0 -> 133.1 mm, vias 5 -> 3
- net unconnected-(SW5-B-Pad2): track 0.00 -> 19.9 mm, vias 0 -> 2
- net (no net): track 45.3 -> 42.0 mm
- net unconnected-(Brd1-VCC-Pad2): track 0.00 -> 3.32 mm
- net GND: vias 61 -> 62
- net 3.3V: vias 5 -> 4
Other:
- board size 100 x 61 mm -> 100 x 75 mm

Commit message: update
Parts:
- removed C4, C5, C6: 0.1uF, project_fp:C_0805_2012Metric_Pad1.15x1.40mm_HandSolder
- removed C7: 1uF, project_fp:C_0805_2012Metric_Pad1.15x1.40mm_HandSolder
- removed CC1, CC2: 5.1k, project_fp:R_0805_2012Metric_Pad1.20x1.40mm_HandSolder
- removed G1, G2: jumper, project_fp:SolderJumper-2_P1.3mm_Open_TrianglePad1.0x1.5mm
- removed HPTRS1, HPTRS2, HPTRS3, HPTRS4 (x2): 3.5MM JACK, project_fp:35RAPC3BH3
- removed IC1: TMUX4053DYYR, SamacSys_Parts:SOP50P326X110-16N
- removed IC2: SN74LVC245ARGYR, SamacSys_Parts:SN74LVC541ARGYR
- removed IC3: TMUX4052BQBR, SamacSys_Parts:TMUX4052BQBR
- removed IC4: TMUX4053BQBR, SamacSys_Parts:TMUX4053BQBR
- removed J1: header, project_fp:PinHeader_1x02_P2.54mm_Vertical_W_CUT
- removed MIC1: SPH0655LM4H-1, project_fp:SPH0655LM4H-1_KNO
- removed Q1, Q2: IRLML6344TRPBF, SamacSys_Parts:SOT95P237X112-3N
- removed R1, R10, R2, R3, R4, R5, R9: 100 ohm, project_fp:R_0805_2012Metric_Pad1.20x1.40mm_HandSolder
- removed R12, R8: 2.2k ohm - 2200 ohm, project_fp:R_0805_2012Metric_Pad1.20x1.40mm_HandSolder
- removed R13, R14, R15, R6: 10k, project_fp:R_0805_2012Metric_Pad1.20x1.40mm_HandSolder
- removed R16: 0 ohm, project_fp:R_0805_2012Metric_Pad1.20x1.40mm_HandSolder
- removed R17, R18, R19, R20: 49.9 ohm, project_fp:R_0805_2012Metric_Pad1.20x1.40mm_HandSolder
- removed R21, R23, R24, R25: 6.8k, project_fp:R_0805_2012Metric_Pad1.20x1.40mm_HandSolder
- removed S1: PEC12R-2220F-S0024, project_fp:XDCR_PEC12R-2220F-S0024
- removed TDM1 (x2): header, project_fp:T-DSP_Expansion_Header_2x10_ALT_GND
- removed U1: Teensy 4.1 - DEVKIT, project_fp:Teensy41_mod2
- removed U2: ESP32-DevKitC - DEVKIT, project_fp:ESP32-DevKitC_NO_COURTYARD
- removed USBA1: USB A Host - TE 292303-5, project_fp:TE_292303-5_USB_A
- removed USBB1: USB B Device (Optional) - B1HSxx, project_fp:USB_B_OST_USB-B1HSxx_Horizontal
- removed USBC1: USB C Device - USB4085-GF-A, project_fp:GCT_USB4085-GF-A_REVA4
- removed USB_IN1, USB_THRU1: header, project_fp:USB_IN1
- removed board_outline1: TAC5212 Module, project_fp:audio_module_board_outline_50x34.5_d1_mod
- removed board_outline2: board_outline, project_fp:audio_project_board_outline_100x75
Routing:
- net 2_OUT2: track 62.8 -> 0.00 mm
- net 5_IN2: track 49.1 -> 0.00 mm
- net Net-(IC1-S2B): track 47.3 -> 0.00 mm
- net HOST_5V: track 43.1 -> 3.91 mm
- net 4_BCLK2: track 38.0 -> 0.00 mm, vias 1 -> 0
- net HOST_D1-: track 35.5 -> 0.00 mm
- net /OUTPUTA: track 81.0 -> 46.2 mm, vias 1 -> 0
- net Net-(IC1-S1B): track 33.8 -> 0.00 mm
- net Net-(board_outline1-IN1P): track 33.2 -> 0.00 mm
- net HOST_D1+: track 32.4 -> 0.00 mm
- net unconnected-(SW5-B-Pad2): track 19.9 -> 0.00 mm, vias 2 -> 0
- net 35_TX8_RESET: track 79.9 -> 63.3 mm, vias 2 -> 0
- net TEENSY_LED: track 15.8 -> 0.00 mm, vias 1 -> 0
- net 3_LRCLK2: track 12.1 -> 0.00 mm, vias 1 -> 0
- net 5V: track 133.1 -> 121.4 mm, vias 3 -> 0
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Other:
- board size 100 x 75 mm -> 80 x 62 mm
