File: audio_back_plane_35_rca.kicad_pcb (KiCad board)
At the start: 4 copper layers, 120 x 100 mm, 106 parts, among them J1 PJRAS2X1S01X, J2 PJRAS2X1S01X, J4 Conn_01x08, U1 Teensy 4.1 - DEVKIT, U10 SN74LVC1T45DBV, U11 SN74LVC1T45DBV, U12 SN74LVC1T45DBV, U13 SN74LVC1T45DBV, U14 Single Buffer - 74LVC1G125GV,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, U15 Single Buffer - 74LVC1G125GV,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

Commit message: update
Parts:
- removed C16, C17, C18, C19, C2, C20, C26, C27, C28, C5: 0.1uF, project_fp:C_0805_2012Metric_Pad1.15x1.40mm_HandSolder
- removed IN1: jumper, project_fp:SolderJumper-3_P_12_BRIDGED
- removed J4: Conn_01x08, Connector_PinHeader_2.54mm:PinHeader_1x08_P2.54mm_Vertical
- removed MIC1: SPH0645LM4H-B, project_fp:SPH0655LM4H-1_KNO
- removed MIC2: SPH0655LM4H-1, project_fp:SPH0655LM4H-1_KNO
- removed OUTA1, OUTB1, OUTC1, OUTD1: jumper, project_fp:SolderJumper-3_P_23_BRIDGED
- removed R16, R17, R18, R19, R35: 49.9 ohm, project_fp:R_0805_2012Metric_Pad1.20x1.40mm_HandSolder
- removed R20, R30, R31: 0 ohm, project_fp:R_0805_2012Metric_Pad1.20x1.40mm_HandSolder
- removed U10, U11, U12, U13, U9: SN74LVC1T45DBV, Package_TO_SOT_SMD:SOT-23-6
- removed U14, U7, U8: Single Buffer - 74LVC1G125GV,125 - SOT-23-5/SC-74A/SOT-753, Package_TO_SOT_SMD:SOT-23-5
- added C4: 0.1uF, project_fp:C_0805_2012Metric_Pad1.15x1.40mm_HandSolder, F.Cu at (119.5, 141.0)
- added D3: HEADER, Connector_PinHeader_2.54mm:PinHeader_2x02_P2.54mm_Vertical, F.Cu at (213.0, 183.5)
- added R14: 49.9 ohm, project_fp:R_0805_2012Metric_Pad1.20x1.40mm_HandSolder, F.Cu at (122.0, 155.0)
- added R15: 49.9 ohm, project_fp:R_0805_2012Metric_Pad1.20x1.40mm_HandSolder, F.Cu at (124.5, 155.0)
- added R32: 49.9 ohm, project_fp:R_0805_2012Metric_Pad1.20x1.40mm_HandSolder, F.Cu at (127.0, 155.0)
- added R33: 49.9 ohm, project_fp:R_0805_2012Metric_Pad1.20x1.40mm_HandSolder, F.Cu at (117.0, 155.0)
- added R34: 49.9 ohm, project_fp:R_0805_2012Metric_Pad1.20x1.40mm_HandSolder, F.Cu at (119.5, 155.0)
- added R36: 49.9 ohm, project_fp:R_0805_2012Metric_Pad1.20x1.40mm_HandSolder, F.Cu at (122.0, 141.0)
- added R37: 49.9 ohm, project_fp:R_0805_2012Metric_Pad1.20x1.40mm_HandSolder, F.Cu at (124.5, 141.0)
- added U3: SN74LVC245APW, Package_SO:TSSOP-20_4.4x6.5mm_P0.65mm, F.Cu at (122.0, 148.0)
- added USB_THRU1: header, project_fp:USB_IN1, F.Cu at (169.4, 115.0)
- G2: moved to B.Cu
- U1: footprint project_fp:Teensy41_mod -> project_fp:Teensy41_mod3
- moved C7 22.0 mm to (193.5, 115.5), turned to 0 degrees
- moved R9 21.4 mm to (157.5, 181.5), turned to -90 degrees
- moved R21 15.7 mm to (194.5, 130.0)
- moved R11 14.6 mm to (171.5, 176.0)
- moved RLED1 14.1 mm to (169.5, 110.5), turned to -90 degrees
- moved PWR1 12.8 mm to (173.0, 110.0), turned to 90 degrees
- moved C8 12.4 mm to (194.5, 127.5), turned to 180 degrees
- moved R23 12.3 mm to (194.5, 132.5)
- moved R29 10.3 mm to (206.0, 123.2)
- moved D23 9.94 mm to (194.0, 122.0), turned to 0 degrees
- moved R24 9.82 mm to (194.5, 125.0), turned to 180 degrees
- moved C21 9.18 mm to (167.0, 183.5), turned to 180 degrees
- moved C11 9.16 mm to (200.5, 128.0)
- moved R26 7.92 mm to (206.0, 132.5), turned to 180 degrees
- moved G2 7.00 mm to (175.5, 110.5)
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- renumbered TDM4 to TDM1, TDM3 to TDM2
Connections:
- PWR1 pad 1: unconnected-(PWR1-K-Pad1) -> GND
- RLED1 pad 2: unconnected-(RLED1-Pad2) -> 5V
- TDM1 pad 15: SDA_C -> SDA_D
- TDM1 pad 17: SCL_C -> SCL_D
- TDM2 pad 15: SDA_D -> SDA_C
- TDM2 pad 17: SCL_D -> SCL_C
- TDM2 pad 7: 8_IN1+ -> 6_OUT1D+
- TDM2 pad 9: 7_OUT1A+ -> 9_OUT1C+
- U1 pad 2: unconnected-(U1-0_RX1_CRX2_CS1-Pad2) -> MIDI_RX
- U1 pad 3: unconnected-(U1-1_TX1_CTX2_MISO1-Pad3) -> MIDI_TX_T
- USBC1 pad A4: 5VIN2 -> 5V
- USBC1 pad A9: 5VIN2 -> 5V
- USBC1 pad B4: 5VIN2 -> 5V
- USBC1 pad B9: 5VIN2 -> 5V
- board_outline1 pad 41: unconnected-(board_outline1-GPIO2-Pad41) -> Net-(D3-Pin_2)
- board_outline1 pad 42: unconnected-(board_outline1-GPO1-Pad42) -> Net-(D3-Pin_3)
Routing:
- net ESP32_IO12_SPI_MISO: track 0.00 -> 71.3 mm
- net ESP32_IO13_SPI_MOSI: track 0.00 -> 65.9 mm
- net 4_BCLK2: track 0.00 -> 46.6 mm
- net USB_SHIELD: track 0.00 -> 43.1 mm
- net MIDI_IN_5: track 0.00 -> 42.0 mm
- net LRCK1: track 0.00 -> 38.3 mm
- net BCLK1: track 0.00 -> 36.5 mm
- net ESP32_IO33_SPI_CS: track 0.00 -> 20.9 mm
- net TEENSY_LED: track 0.00 -> 20.6 mm
- net MIDI_RX: track 0.00 -> 19.6 mm
- net Net-(U1-33_MCLK2): track 0.00 -> 19.0 mm
- net MCLK1: track 0.00 -> 18.8 mm
- net 3_LRCLK2: track 0.00 -> 18.7 mm
- net 35_TX8_RESET: track 0.00 -> 18.6 mm
- net MIDI_IN_4: track 0.00 -> 17.5 mm
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
Commit message: update
Parts:
- added JP1: Jumper_2_Open, project_fp:jumper_slice_disconnected, F.Cu at (165.0, 197.0)
- added JP2: Jumper_2_Open, project_fp:jumper_slice_disconnected, F.Cu at (171.0, 197.0)
- D2, D5: footprint project_fp:LED_4691 -> project_fp:SK6812-32228SMD-Reverse-Mount
- moved TDM1 2.00 mm to (102.0, 132.0)
- moved TDM2 2.00 mm to (102.0, 169.0)
- moved C1 1.00 mm to (171.0, 189.0)
- moved C3 1.00 mm to (165.0, 189.0)
- moved R12 1.00 mm to (171.0, 195.0)
- moved R13 1.00 mm to (165.0, 195.0)
- moved U15 1.00 mm to (171.0, 192.0)
- moved U16 1.00 mm to (165.0, 192.0)
Connections:
- D2 pad 1: 5V -> Net-(D2-VDD)
- D2 pad 2: ESP32_LED+ -> 5V
- D2 pad 3: GND -> ESP32_LED+
- D2 pad 4: Net-(D2-DIN) -> GND
- D5 pad 1: 5V -> Net-(D5-DIN)
- D5 pad 2: TEENSY_LED+ -> 5V
- D5 pad 3: GND -> TEENSY_LED+
- D5 pad 4: Net-(D5-DIN) -> GND
- R12 pad 1: Net-(D2-DIN) -> Net-(D2-VDD)
Routing:
- net TEENSY_LED: track 20.6 -> 0.00 mm
- net 9_OUT1C+: track 11.8 -> 0.00 mm
- net 7_OUT1A+: track 10.1 -> 2.02 mm
- net GND: track 0.00 -> 4.92 mm
- net Net-(D2-VDD): track 0.00 -> 4.42 mm
- net 6_OUT1D+: track 4.38 -> 0.00 mm
- net Net-(D2-DIN): track 3.89 -> 0.00 mm
- net 8_IN1+: track 6.87 -> 9.98 mm
- net Net-(U16-Y): track 2.11 -> 0.00 mm
- net Net-(U15-Y): track 2.11 -> 0.00 mm
- net TEENSY_LED+: track 0.00 -> 1.86 mm
- net ESP32_LED+: track 0.00 -> 1.86 mm
- net ESP32_IO13_SPI_MOSI: track 65.9 -> 65.1 mm
- net Net-(D5-DIN): track 3.89 -> 4.42 mm

Commit message: update
Parts:
- removed R6: 10k, project_fp:R_0805_2012Metric_Pad1.20x1.40mm_HandSolder
- added R38: 49.9 ohm, project_fp:R_0805_2012Metric_Pad1.20x1.40mm_HandSolder, F.Cu at (164.5, 159.5)
- added R39: 49.9 ohm, project_fp:R_0805_2012Metric_Pad1.20x1.40mm_HandSolder, F.Cu at (164.5, 162.0)
- D3: footprint Connector_PinHeader_2.54mm:PinHeader_2x02_P2.54mm_Vertical -> project_fp:TAC5212_GPIO_PinHeader_2x02_P2.54mm_Vertical
- moved G1 67.6 mm to (189.0, 106.9)
- moved ILI_VCC1 66.2 mm to (210.5, 151.8)
- moved D3 40.6 mm to (213.0, 142.9)
- moved C31 33.2 mm to (201.5, 189.5), turned to 180 degrees
- moved R32 31.1 mm to (129.0, 124.0), turned to 180 degrees
- moved board_outline1 29.9 mm to (157.5, 146.8), turned to 180 degrees
- moved R14 29.3 mm to (129.0, 126.5), turned to 180 degrees
- moved C4 29.0 mm to (144.0, 125.5), turned to 180 degrees
- moved R59 26.7 mm to (185.0, 154.0), turned to 180 degrees
- moved R33 26.4 mm to (129.0, 131.5), turned to 180 degrees
- moved R15 26.4 mm to (129.0, 129.0), turned to 180 degrees
- moved U3 25.9 mm to (142.0, 131.5), turned to 0 degrees
- moved R34 23.0 mm to (129.0, 134.0), turned to 180 degrees
- moved R36 20.7 mm to (129.0, 121.5), turned to 180 degrees
- moved R7 20.6 mm to (185.0, 169.0)
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Connections:
- HPTRS4 pad 3: Net-(HPTRS4-Pad3) -> unconnected-(HPTRS4-Pad3)
- HPTRS4 pad 4: IN2_JACK_DETECT -> Net-(HPTRS4-Pad4)
- J1 pad S1: GND -> unconnected-(J1-PadS1)
- J1 pad T1: Net-(HPTRS4-Pad3) -> unconnected-(J1-PadT1)
- J1 pad T2: IN2_JACK_DETECT -> Net-(HPTRS4-Pad4)
- R14 pad 1: Net-(U3-A5) -> Net-(U3-A3)
- R14 pad 2: LRCK1+ -> BCLK1+
- R15 pad 1: Net-(U3-A6) -> Net-(U3-A4)
- R15 pad 2: BCLK1+ -> LRCK1+
- R32 pad 1: Net-(U3-A8) -> Net-(U3-A1)
- R33 pad 1: Net-(U3-A2) -> Net-(U3-A6)
- R34 pad 1: Net-(U3-A4) -> Net-(U3-A8)
- R36 pad 1: Net-(U3-B1) -> Net-(U3-B5)
- R37 pad 1: Net-(U3-B3) -> Net-(U3-B7)
- TDM1 pad 15: SDA_D -> SDA0
- TDM1 pad 17: SCL_D -> SCL0
- TDM2 pad 15: SDA_C -> SDA0
- TDM2 pad 17: SCL_C -> SCL0
- U1 pad 26: unconnected-(U1-34_RX8-Pad26) -> 34_RX8_RESET2
- U1 pad 8: 6_OUT1D -> Net-(U1-6_OUT1D)
- U1 pad 9: 7_OUT1A -> Net-(U1-7_RX2_OUT1A)
- U3 pad 10: unconnected-(U3-GND-Pad10) -> GND
- U3 pad 11: MCLK1 -> 9_OUT1C
- U3 pad 12: GND -> Net-(U3-B7)
- U3 pad 13: BCLK1 -> 7_OUT1A
- U3 pad 14: LRCK1 -> Net-(U3-B5)
- U3 pad 15: 9_OUT1C -> LRCK1
- U3 pad 16: Net-(U3-B3) -> BCLK1
- U3 pad 17: 7_OUT1A -> GND
- U3 pad 18: Net-(U3-B1) -> MCLK1
- U3 pad 2: 8_IN1 -> Net-(U3-A1)
- U3 pad 3: Net-(U3-A2) -> GND
- U3 pad 4: 6_OUT1D -> Net-(U3-A3)
- U3 pad 6: Net-(U3-A5) -> 8_IN1
- U3 pad 8: GND -> 6_OUT1D
Routing:
- net Net-(HPTRS4-Pad4): track 0.00 -> 137.3 mm
- net MCLK1+: track 0.00 -> 125.1 mm, vias 0 -> 3
- net 34_RX8_RESET2: track 0.00 -> 124.3 mm, vias 0 -> 1
- net (no net): track 0.00 -> 101.7 mm
- net 35_TX8_RESET: track 18.6 -> 111.8 mm, vias 0 -> 2
- net Net-(HPTRS1-Pad3): track 0.00 -> 85.0 mm
- net Net-(HPTRS1-Pad4): track 0.00 -> 83.0 mm
- net TEENSY_LED+: track 1.86 -> 78.9 mm, vias 0 -> 1
- net SCL0: track 0.00 -> 75.0 mm, vias 0 -> 1
- net 53_T_PROG: track 3.57 -> 74.8 mm
- net 2_OUT2: track 0.00 -> 70.6 mm, vias 0 -> 1
- net 5V: track 3.53 -> 73.6 mm, vias 0 -> 7
- net 7_OUT1A: track 0.00 -> 69.5 mm, vias 0 -> 3
- net ESP32_LED+: track 1.86 -> 71.3 mm, vias 0 -> 1
- net ESP32_EN: track 0.00 -> 68.1 mm
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- added copper zone on B.Cu, net 3.3V
- added copper zone on F.Cu, net 3.3V
- added copper zone on In1.Cu, net 3.3V
- added copper zone on B.Cu, net GND
- added copper zone on F.Cu, net GND
- added copper zone on In1.Cu, net GND
- added copper zone on In4.Cu, net GND
Other:
- copper layers 4 -> 6

Commit message: update
Parts:
- moved JP2 0.50 mm to (171.0, 196.5)
Connections:
- HPTRS4 pad 3: unconnected-(HPTRS4-Pad3) -> Net-(HPTRS4-Pad3)
- J1 pad S1: unconnected-(J1-PadS1) -> Net-(HPTRS4-Pad3)
- J1 pad T1: unconnected-(J1-PadT1) -> GND
Routing:
- net 5V: track 73.6 -> 363.4 mm, vias 7 -> 9
- net Net-(HPTRS4-Pad3): track 0.00 -> 103.1 mm
- net (no net): track 101.7 -> 0.00 mm
- net SDA0: track 66.9 -> 127.7 mm, vias 1 -> 2
- net SCL0: track 75.0 -> 133.9 mm
- net GND: track 21.4 -> 75.0 mm, vias 4 -> 10
- net 35_TX8_RESET: track 111.8 -> 157.5 mm, vias 2 -> 3
- net ESP32_IO0: track 51.8 -> 93.6 mm
- net /ESP32_IO1: track 0.00 -> 41.6 mm, vias 0 -> 1
- net /SWITCH: track 14.2 -> 54.2 mm, vias 0 -> 2
- net /ESP32_IO3: track 0.00 -> 38.2 mm
- net Net-(ILI1-CS): track 0.00 -> 34.3 mm
- net /OUTPUTB: track 17.7 -> 49.5 mm, vias 0 -> 1
- net ESP32_EN: track 68.1 -> 98.8 mm
- net Net-(GPI1-Pin_2): track 0.00 -> 23.9 mm, vias 0 -> 2
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- added copper zone on In3.Cu, net 3.3V
- removed copper zone on B.Cu, net 3.3V
- removed copper zone on F.Cu, net 3.3V
- removed copper zone on In1.Cu, net 3.3V
- removed copper zone on In2.Cu, net 3.3V

Commit message: update
Parts:
- removed C4: 0.1uF, project_fp:C_0805_2012Metric_Pad1.15x1.40mm_HandSolder
- removed JP1, JP2: Jumper_2_Open, project_fp:jumper_slice_disconnected
- removed R12, R13: 0 ohm, project_fp:R_0805_2012Metric_Pad1.20x1.40mm_HandSolder
- removed R14, R15, R32, R33, R34, R36, R37: 49.9 ohm, project_fp:R_0805_2012Metric_Pad1.20x1.40mm_HandSolder
- removed U15, U16: Single Buffer - 74LVC1G125GV,125 - SOT-23-5/SC-74A/SOT-753, Package_TO_SOT_SMD:SOT-23-5
- removed U3: SN74LVC245APW, Package_SO:TSSOP-20_4.4x6.5mm_P0.65mm
- added C17: 0.1uF, project_fp:C_0805_2012Metric_Pad1.15x1.40mm_HandSolder, F.Cu at (169.5, 194.5)
- added C18: 10uF, project_fp:C_0805_2012Metric_Pad1.15x1.40mm_HandSolder, F.Cu at (172.0, 194.5)
- added C19: 0.1uF, project_fp:C_0805_2012Metric_Pad1.15x1.40mm_HandSolder, F.Cu at (155.5, 133.5)
- added C20: 0.1uF, project_fp:C_0805_2012Metric_Pad1.15x1.40mm_HandSolder, F.Cu at (155.5, 115.5)
- added IC1: 74HCT2G125DC,125, project_fp:SOP50P310X100-8N, F.Cu at (165.5, 195.0)
- added U21: SN74LVC2G125DCTR, project_fp:SOP65P400X130-8N, F.Cu at (155.5, 118.5)
- added U22: SN74LVC2G125DCTR, project_fp:SOP65P400X130-8N, F.Cu at (155.5, 130.5)
- added U23: SN74LVC2G125DCTR, project_fp:SOP65P400X130-8N, F.Cu at (155.5, 124.5)
- added U24: SN74LVC2G125DCTR, project_fp:SOP65P400X130-8N, F.Cu at (155.5, 136.5)
- D2, D5: footprint project_fp:SK6812-32228SMD-Reverse-Mount -> project_fp:SK6812-32228SMD-Reverse-Mount_mod
- moved C3 68.2 mm to (155.5, 121.5)
- moved C1 63.4 mm to (155.5, 127.5)
- moved board_outline1 40.2 mm to (119.8, 133.0), turned to -90 degrees
- moved D2 0.50 mm to (171.0, 199.5)
- moved D5 0.50 mm to (165.0, 199.5)
Connections:
- C1 pad 1: 5V -> 3.3V
- C3 pad 1: 5V -> 3.3V
- D1 pad 1: ESP32_LED+ -> ESP32_LED_OUT
- D1 pad 2: TEENSY_LED+ -> TEENSY_LED_OUT
- D1 pad 4: 5V -> LED_PWR
- D2 pad 1: Net-(D2-VDD) -> ESP32_LED+
- D2 pad 3: ESP32_LED+ -> ESP32_LED_OUT
- D5 pad 1: Net-(D5-DIN) -> TEENSY_LED+
- D5 pad 3: TEENSY_LED+ -> TEENSY_LED_OUT
- TDM1 pad 11: BCLK1+ -> BCLK1+TDM1
- TDM1 pad 13: LRCK1+ -> LRCK1+TDM1
- TDM1 pad 19: MCLK1+ -> MCLK1+TDM1
- TDM1 pad 7: 8_IN1+ -> 8_IN1
- TDM2 pad 11: BCLK1+ -> BCLK1+TDM2
- TDM2 pad 13: LRCK1+ -> LRCK1+TDM2
- TDM2 pad 19: MCLK1+ -> MCLK1+TDM2
- TDM2 pad 7: 6_OUT1D+ -> 9_OUT1C_INPUT
- TDM2 pad 9: 9_OUT1C+ -> 6_OUT1D+
- U1 pad 11: 9_OUT1C -> 9_OUT1C_INPUT
- board_outline1 pad 11: BCLK1 -> BCLK1+TDM1
- board_outline1 pad 13: LRCK1 -> LRCK1+TDM1
- board_outline1 pad 19: MCLK1 -> MCLK1+TDM1
- board_outline1 pad 7: 7_OUT1A -> 7_OUT1A+
Routing:
- net 5V: track 363.4 -> 149.5 mm, vias 9 -> 4
- net 35_TX8_RESET: track 157.5 -> 19.8 mm, vias 3 -> 0
- net Net-(HPTRS4-Pad4): track 137.3 -> 0.00 mm
- net 34_RX8_RESET2: track 122.1 -> 0.00 mm, vias 1 -> 0
- net MCLK1+: track 120.1 -> 0.00 mm, vias 3 -> 0
- net MCLK1+TDM2: track 0.00 -> 114.5 mm, vias 0 -> 1
- net Net-(HPTRS4-Pad3): track 103.1 -> 0.00 mm
- net BCLK1+TDM2: track 0.00 -> 94.1 mm, vias 0 -> 1
- net SDA0: track 127.7 -> 37.9 mm, vias 2 -> 0
- net 9_OUT1C_INPUT: track 0.00 -> 87.9 mm, vias 0 -> 1
- net SCL0: track 133.9 -> 46.9 mm, vias 1 -> 0
- net Net-(HPTRS1-Pad3): track 85.0 -> 0.00 mm
- net Net-(HPTRS1-Pad4): track 83.0 -> 0.00 mm
- net LRCK1+TDM2: track 0.00 -> 81.6 mm, vias 0 -> 1
- net MCLK1+TDM1: track 0.00 -> 81.6 mm, vias 0 -> 2
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
Commit message: update
Routing:
- net Net-(board_outline1-OUTP): track 0.00 -> 47.2 mm
- net SDA0: track 37.9 -> 74.2 mm
- net Net-(1/4-PHONE1-PadRN): track 0.00 -> 35.4 mm
- net Net-(board_outline1-IN2P): track 0.00 -> 34.5 mm
- net Net-(board_outline1-OUT2P): track 0.00 -> 34.3 mm
- net Net-(1/4-PHONE1-PadTN): track 0.00 -> 32.9 mm
- net Net-(board_outline1-IN1P): track 0.00 -> 32.0 mm
- net 9_OUT1C_INPUT: track 87.9 -> 56.1 mm, vias 1 -> 0
- net 7_OUT1A+: track 30.5 -> 58.7 mm, vias 1 -> 2
- net 35_TX8_RESET: track 19.8 -> 47.1 mm, vias 0 -> 1
- net 5V: track 149.5 -> 175.4 mm
- net 8_IN1: track 81.8 -> 59.4 mm, vias 1 -> 2
- net SCL0: track 46.9 -> 38.2 mm
- net BCLK1+TDM2: track 94.1 -> 87.7 mm, vias 1 -> 3
- net DEVICE_D1+: track 44.8 -> 38.5 mm
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- added copper zone on In2.Cu, net GND
- added copper zone on In3.Cu, net GND
- added copper zone on In5.Cu, net GND
- added copper zone on In6.Cu, net GND
Other:
- copper layers 6 -> 8
- board text added: "KiCad 8-Layer Stackup: F.Cu - TOP: Components, ANALOG routes to jacks, ground fill In1.Cu - GND: Solid ground plane In2.Cu - SIG1: TDM/high-speed digital, ground fill In3.Cu - GND: Solid ground plane (isolation!) In4.Cu - SIG2: More TDM/digital signals, ground fill In5.Cu - PWR: Power planes (3.3V/5V) In6.Cu - GND: Solid ground plane B.Cu - BOTTOM: Components, ANALOG routes to jacks, ground fill"
