File: audio_back_plane_35_rca.kicad_sch (KiCad schematic)
At the start: 96 parts, among them IC1 TMUX4053DYYR, IC2 SN74LVC245ARGYR, IC3 TMUX4052BQBR, IC4 TMUX4053BQBR, IC5 TMUX4053DYYR, J1 header, Q1 IRLML6344TRPBF, Q2 IRLML6344TRPBF, SW1 RotaryEncoder_Switch_MP, SW2 TL1105WF160Q - 3.15mm actuator, SW3 TL1105WF160Q - 3.15mm actuator, SW4 TL1105WF160Q - 3.15mm actuator, SW5 TL1105WF160Q - 3.15mm actuator, SW6 TL1105WF160Q - 3.15mm actuator, U1 Teensy 4.1 - DEVKIT, U2 ESP32-DevKitC - DEVKIT, U3 TFT_320x240, U4 EN11-HSM1AF15

Commit message: update
Parts:
- removed HPTRS3: 3.5MM JACK, project_fp:35RAPC3BH3, symbol 35RAPC3BH3:AudioJack3_SwitchTR
- removed IC1: TMUX4053DYYR, SOP50P326X110-16N, symbol SamacSys_Parts:TMUX4053DYYR_MOD
- removed IC4: TMUX4053BQBR, TMUX4053BQBR, symbol SamacSys_Parts:TMUX4053BQBR
- removed Q1, Q2: IRLML6344TRPBF, SOT95P237X112-3N, symbol SamacSys_Parts:IRLML6344TRPBF
- removed R21, R23, R24, R25: 6.8k, project_fp:R_0805_2012Metric_Pad1.20x1.40mm_HandSolder, symbol Device:R
- added J2, J5: NMJ6HFD2-AU, Connector_Audio:Jack_6.35mm_Neutrik_NMJ6HFD2-AU_Horizontal, symbol Connector_Audio:NMJ6HFD2-AU
- added J3, J6: Conn_Coaxial_x2, project_fp:PJRAS2X1_NOT-VERIFIED, symbol Connector:Conn_Coaxial_x2
- added J4: Conn_01x08, Connector_PinHeader_2.54mm:PinHeader_1x08_P2.54mm_Vertical, symbol Connector_Generic:Conn_01x08
- D1, D4: footprint project_fp:PinHeader_1x04_P1.00mm_Vertical_WS2812_LED_mod -> project_fp:PinHeader_1x04_P2.54mm_Vertical; now fitted
- IC3, USBB1, USB_IN1, USB_THRU1: now left out of the parts list
- S1: now not fitted
- board_outline2: footprint project_fp:audio_project_board_outline_100x75 -> project_fp:audio_project_board_outline_125x75
Connections:
- net GND: no longer HPTRS2.1
- net at HPTRS4.3: no longer board_outline1.31 (IN1M)
- new net: MIC1.4 (LRCLK-WS-FS), MIC2.4 (LRCLK-WS-FS), board_outline1.40 (GPIO1)
- now unconnected: MIC1.4 (LRCLK-WS-FS), MIC2.4 (LRCLK-WS-FS)
Other:
- moved on the sheet: Brd1, C1, C3, D10, D11, D12, D13, D14, D15, D16, D17, D18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

Commit message: update
Parts:
- removed C4, C6: 0.1uF, project_fp:C_0805_2012Metric_Pad1.15x1.40mm_HandSolder, symbol TEENSY_4.0_ESP32_AUDIO-rescue:C_Small-Device
- removed HPTRS2: 3.5MM JACK, project_fp:35RAPC3BH3, symbol 35RAPC3BH3:AudioJack3_SwitchTR
- removed J1: header, project_fp:PinHeader_1x02_P2.54mm_Vertical_W_CUT, symbol Connector_Generic:Conn_02x02_Odd_Even
- removed J5: NMJ6HFD2-AU, Connector_Audio:Jack_6.35mm_Neutrik_NMJ6HFD2-AU_Horizontal, symbol Connector_Audio:NMJ6HFD2-AU
- added 1/4-PHONE1: NMJ6HFD2-AU, project_fp:Jack_6.35mm_Neutrik_NMJ6HCD3_Horizontal, symbol NMJ6HCD3:AudioPlug3
- added BAT1: Battery Cell - TE 1775485-1, project_fp:TE_1775485-1_BATTERY, symbol Device:Battery_Cell
- added C11, C16, C17, C18, C19, C20, C23, C24, C25, C26, C27, C28, C29, C30, C8: 0.1uF, project_fp:C_0805_2012Metric_Pad1.15x1.40mm_HandSolder, symbol Device:C_Small
- added C21, C22, C31, C32: 0.1uF, project_fp:C_0805_2012Metric_Pad1.15x1.40mm_HandSolder, symbol TEENSY_4.0_ESP32_AUDIO-rescue:C_Small-Device
- added D23: Diode - 1N4148, project_fp:D_SOD-123, symbol Diode:1N4148
- added H1, H2, H3, H6: MountingHole_Pad, MountingHole:MountingHole_3.2mm_M3_DIN965_Pad, symbol Mechanical:MountingHole_Pad
- added IN1: jumper, project_fp:SolderJumper-3_P_12_BRIDGED, symbol Jumper:SolderJumper_3_Bridged12
- added MIDI_IN_1, MIDI_OUT_1: 3.5mm TRS - 35RAPC3BH3, project_fp:35RAPC3BH3, symbol project_lil_2:35RAPC4BH3
- added MIDI_IO1: header, project_fp:MIDI_IO1, symbol Connector_Generic:Conn_02x06_Odd_Even
- added MIDI_OT1, MIDI_OT2: jumper, project_fp:SolderJumper-3_P1.3mm_Bridged2Bar12_Pad1.0x1.5mm_NumberLabels, symbol Jumper:SolderJumper_3_Bridged12
- added OUTA1, OUTB1, OUTC1, OUTD1: jumper, project_fp:SolderJumper-3_P_23_BRIDGED, symbol project_lil_2:SolderJumper_3_Bridged23
- added PWR1: LED_1206, Diode_SMD:D_1210_3225Metric_Pad1.42x2.65mm_HandSolder, symbol Device:LED
- added R21, R25, R40: 0ohm, project_fp:R_0805_2012Metric_Pad1.20x1.40mm_HandSolder, symbol Device:R
- added R22, R24, R27, R28: 220 ohm, project_fp:R_0805_2012Metric_Pad1.20x1.40mm_HandSolder, symbol Device:R_Small
- added R23: 1.5k, project_fp:R_0805_2012Metric_Pad1.20x1.40mm_HandSolder, symbol Device:R_Small
- added R26, R29: 47 ohm, project_fp:R_0805_2012Metric_Pad1.20x1.40mm_HandSolder, symbol Device:R_Small
- added R30, R31: 0 ohm, project_fp:R_0805_2012Metric_Pad1.20x1.40mm_HandSolder, symbol Device:R
- added R32, R33, R34, R35: 49.9 ohm, project_fp:R_0805_2012Metric_Pad1.20x1.40mm_HandSolder, symbol Device:R
- added R63: 470 ohm, project_fp:R_0805_2012Metric_Pad1.20x1.40mm_HandSolder, symbol Device:R_Small
- added RLED1: led, project_fp:R_0805_2012Metric_Pad1.20x1.40mm_HandSolder, symbol Device:R
- added SW7, SW8: SW_SPST, project_fp:SW_Tactile_SPST_Angled_PTS645Vx39-2LFS, symbol Switch:SW_SPST
- added TDM2, TDM3, TDM4: header, project_fp:T-DSP_Expansion_Header_2x10_ALT_GND, symbol project_lil_2:TDM_HEADER_Conn_02x10_Odd_Even
- added T_PROG1: header, project_fp:T_PROG1_PinHeader_1x03_P2.54mm_Vertical, symbol Connector_Generic:Conn_01x03
- added U10, U11, U12, U13, U9: SN74LVC1T45DBV, Package_TO_SOT_SMD:SOT-23-6, symbol Logic_LevelTranslator:SN74LVC1T45DBV
- added U14, U7, U8: Single Buffer - 74LVC1G125GV,125 - SOT-23-5/SC-74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, Package_TO_SOT_SMD:SOT-23-5, symbol project_lil_2:SN74LVC1G125
- added U5: Optoisolators - H11L1SM - 6-SMD, Gull Wing, project_fp:IC_H11L1SM, symbol Isolator:H11L1
- added U6: Dual Buffer - 74HCT2G17GW,125 - SOT-363_SC-70-6, project_fp:SOT-363_SC-70-6, symbol project_lib:74HCT2G34
- Brd1, C1, C3, D10, D11, D12, D13, D14, D15, D16, D17, D18, D19, D2, D20, D21, D22, D3, D5, D6, D7, D8, D9, IC2, R11, R7, SW1, SW2, SW3, SW4, TDM1, U4: now not fitted
- HPTRS4: Label IN2 -> IN1
- J3: value Conn_Coaxial_x2 -> RCA-IN
- J6: value Conn_Coaxial_x2 -> RCA-OUT
- MIC1: value SPH0655LM4H-1 -> SPH0645LM4H-B
- R16: value 0 ohm -> 49.9 ohm
- R20: value 49.9 ohm -> 0 ohm
- SW5: value TL1105WF160Q - 3.15mm actuator -> SW_SPST; footprint project_fp:Tactile_Switch_4.54.5MM -> project_fp:SW_Tactile_SPST_Angled_PTS645Vx39-2LFS
- SW6: footprint project_fp:Tactile_Switch_4.54.5MM -> project_fp:SW_Tactile_SPST_Angled_PTS645Vx39-2LFS
- U1: footprint project_fp:Teensy41_mod2 -> project_fp:Teensy41_mod
- board_outline2: footprint project_fp:audio_project_board_outline_125x75 -> project_fp:audio_project_board_outline_100x120
Connections:
- net 12V: now also TDM2.5 (12V), TDM3.5 (12V), TDM4.5 (12V)
- net 3.3V: now also R21.2, R40.2, R63.1
- net 32_OUT1B: now also U13.3 (A)
- net 34_RX8_RESET2: now also TDM2.2 (HELD_LOW), TDM3.2 (HELD_LOW), TDM4.2 (HELD_LOW)
- net 35_TX8_RESET: now also TDM2.1 (HELD_HIGH), TDM3.1 (HELD_HIGH), TDM4.1 (HELD_HIGH)
- net 53_T_PROG: now also SW5.1 (A), C21.1, T_PROG1.1 (Pin_1)
- net 54_ON_OFF: now also SW6.1 (A), C22.1, T_PROG1.3 (Pin_3)
- net 5V: now also R25.2, R27.2, R29.2, TDM2.3 (5V), TDM3.3 (5V), TDM4.3 (5V)
- net 6_OUT1D: now also U11.3 (A)
- net 7_OUT1A: now also U10.3 (A)
- net 7_OUT1A+: now also R16.1, TDM1.9 (DSP_DATA_OUT), TDM2.9 (DSP_DATA_OUT), TDM3.9 (DSP_DATA_OUT), TDM4.9 (DSP_DATA_OUT)
- net 8_IN1: now also U9.3 (A)
- net 8_IN1+: now also TDM1.7 (DSP_DATA_IN), R35.1, TDM2.7 (DSP_DATA_IN), TDM3.7 (DSP_DATA_IN), TDM4.7 (DSP_DATA_IN)
- net 9_OUT1C: now also U12.3 (A)
- net BCLK1: now also U14.2 (A)
- net BCLK1+: now also TDM1.11 (BCLK), R31.1, TDM2.11 (BCLK), TDM3.11 (BCLK), TDM4.11 (BCLK); no longer R18.2
- net ESP32_EN: now also C31.1, SW7.2 (B)
- net ESP32_IO0: now also C32.1, SW8.2 (B)
- net GND: now also J3.3 (EXT), J6.3 (EXT), SW5.2 (B), SW6.2 (B), C11.1, C16.2, C17.2, C18.2, C19.2, C20.2, C21.2, C22.2, C23.2, C24.2, C25.2, C26.2, C27.2, C28.2, C29.2, C30.2, C31.2, C32.2, C8.1, IN1.1 (A), MIDI_IN_1.1, MIDI_IO1.10 (Pin_10), MIDI_IO1.12 (Pin_12), MIDI_IO1.2 (Pin_2), MIDI_IO1.4 (Pin_4), MIDI_IO1.6 (Pin_6), MIDI_IO1.8 (Pin_8), MIDI_OUT_1.1, OUTA1.1 (A), OUTB1.1 (A), OUTC1.1 (A), OUTD1.1 (A), R23.1, SW7.1 (A), SW8.1 (A), TDM2.10 (GND), TDM2.12 (GND), TDM2.14 (GND), TDM2.16 (GND), TDM2.18 (GND), TDM2.20 (GND), TDM2.6 (GND), TDM2.8 (GND), TDM3.10 (GND), TDM3.12 (GND), TDM3.14 (GND), TDM3.16 (GND), TDM3.18 (GND), TDM3.20 (GND), TDM3.6 (GND), TDM3.8 (GND), TDM4.10 (GND), TDM4.12 (GND), TDM4.14 (GND), TDM4.16 (GND), TDM4.18 (GND), TDM4.20 (GND), TDM4.6 (GND), TDM4.8 (GND), T_PROG1.2 (Pin_2), U10.2 (GND), U11.2 (GND), U12.2 (GND), U13.2 (GND), U14.1 (OE), U14.3 (GND), U6.2 (GND), U7.1 (OE), U7.3 (GND), U8.1 (OE), U8.3 (GND), U9.2 (GND)
- net IN2_JACK_DETECT: now also J3.1 (IN1)
- net LRCK1: now also U8.2 (A)
- net LRCK1+: now also TDM1.13 (LRCK), R30.1, TDM2.13 (LRCK), TDM3.13 (LRCK), TDM4.13 (LRCK); no longer R19.2
- net MCLK1: now also U7.2 (A)
- net MCLK1+: now also R20.1, TDM1.19 (MCLK), TDM2.19 (MCLK), TDM3.19 (MCLK), TDM4.19 (MCLK); no longer R20.2
- net SCL_C: now also TDM2.17 (SCL), TDM4.17 (SCL)
- net SDA_C: now also TDM2.15 (SDA), TDM4.15 (SDA)
- net SYSTEM_EN: now also TDM2.4 (GND), TDM3.4 (GND), TDM4.4 (GND)
- net T_BUTTON1: no longer SW5.1 (A)
- net T_BUTTON2: no longer SW6.1 (A)
- net at HPTRS4.2: now also board_outline1.29 (IN1P); no longer board_outline1.35 (IN2M)
- net at HPTRS4.3: now also J3.2 (IN2)
- net 9_OUT1C+: now reaches R18.1
- net 9_OUT1C+: no longer TDM1.11 (BCLK)
- net 32_OUT1B+: now reaches R19.1
- net 32_OUT1B+: no longer TDM1.13 (LRCK)
- net 6_OUT1D+: now reaches R17.1
- net 6_OUT1D+: no longer TDM1.9 (DSP_DATA_OUT)
- net at board_outline1.21 (OUTP): now also 1/4-PHONE1.R
- net at board_outline1.25 (OUT2P): now also 1/4-PHONE1.T
- net at R16.2: now also U10.4 (B)
- net at R17.2: now also U11.4 (B)
- net at HPTRS1.2: now also 1/4-PHONE1.RN
- net at HPTRS1.3: now also J6.2 (IN2)
- net at HPTRS1.4: now also J6.1 (IN1)
- net at HPTRS1.5: now also 1/4-PHONE1.TN
- net at U1.50 (VBAT): now also BAT1.1 (+)
- net at U1.52 (GND): now also BAT1.2 (-)
- new net: MIDI_OT2.2 (C), MIDI_OUT_1.2
- new net: MIDI_OT1.2 (C), MIDI_OUT_1.5
- new net: OUTC1.2 (C), U12.5 (DIR)
- new net: IN1.3 (B), OUTA1.3 (B), OUTB1.3 (B), OUTC1.3 (B), OUTD1.3 (B), R63.2
- new net: R30.2, U8.4 (Y)
- new net: C11.2, R25.1, U6.5 (VCC)
- new net: OUTA1.2 (C), U10.5 (DIR)
- new net: D23.1 (K), R22.2, U5.1
- new net: PWR1.2 (A), RLED1.1
- new net: R35.2, U9.4 (B)
- new net: R20.2, U7.4 (Y)
- new net: C8.2, R21.1, R24.2, U5.6
- new net: MIC1.4 (LRCLK-WS-FS), MIC2.4 (LRCLK-WS-FS), board_outline1.40 (GPIO1)
- new net: OUTD1.2 (C), U11.5 (DIR)
- new net: R28.2, U6.6
- new net: R18.2, U12.4 (B)
- new net: IN1.2 (C), U9.5 (DIR)
- new net: R31.2, U14.4 (Y)
- new net: R23.2, U5.5
- new net: R19.2, U13.4 (B)
- new net: OUTB1.2 (C), U13.5 (DIR)
- new net: R26.2, U6.4
- new net 3.3V_BUFFER: C16.1, C17.1, C18.1, C19.1, C20.1, C23.1, C24.1, C25.1, C26.1, C27.1, C28.1, C29.1, C30.1, R40.1, U10.1 (VCCA), U10.6 (VCCB), U11.1 (VCCA), U11.6 (VCCB), U12.1 (VCCA), U12.6 (VCCB), U13.1 (VCCA), U13.6 (VCCB), U14.5 (VCC), U7.5 (VCC), U8.5 (VCC), U9.1 (VCCA), U9.6 (VCCB)
- new net MIDI_IN_4: MIDI_IN_1.2, MIDI_IO1.1 (Pin_1), R22.1
- new net MIDI_IN_5: D23.2 (A), MIDI_IN_1.5, MIDI_IO1.3 (Pin_3), U5.2
- new net MIDI_OUT_4: MIDI_IO1.5 (Pin_5), MIDI_OT2.1 (A), R29.1
- new net MIDI_OUT_5: MIDI_IO1.7 (Pin_7), MIDI_OT1.1 (A), R28.1
- new net MIDI_RX: R24.1, U5.4, U6.3
- new net MIDI_THRU_4: MIDI_IO1.9 (Pin_9), MIDI_OT2.3 (B), R27.1
- new net MIDI_THRU_5: MIDI_IO1.11 (Pin_11), MIDI_OT1.3 (B), R26.1
- new net MIDI_TX_T: U6.1
- new net S-GND: 1/4-PHONE1.S
- new net SCL_D: TDM3.17 (SCL)
- new net SDA_D: TDM3.15 (SDA)
- new net SN: 1/4-PHONE1.SN
- now unconnected: MIC1.4 (LRCLK-WS-FS), MIC2.4 (LRCLK-WS-FS)
- no-connect marks 8 -> 12
Other:
- note added: "3 PIN MIDI"
- note added: "CLOCK DRIVER"
- note added: "Changed to SPH0645LM4H-B for Target use: Voice/audio capture (speech, speakerphone, voice assistants, etc.)"
- note added: "DATA DRIVER"
- note added: "EXPANSION PORTS"
- note added: "MIDI"
- note added: "MIDI HEADER"
- note added: "MIDI IN"
- note added: "MIDI OUT"
- note added: "MIDI THROUGH"
- note added: "MIDI circuit from TeensyMIDIAudio project."
- note added: "MUST VERIFY LINES AND PADS"
- note added: "PLEASE CONFIRM LEFT/RIGHT PINS"
- note added: "https://electronics.stackexchange.com/questions/310899/midi-out-thru-circuit-questions"
- moved on the sheet: HPTRS1, HPTRS4, J3, J6, R9

Commit message: update
Parts:
- removed #SAI1: header, project_fp:IDC-Header_2x10_P2.54mm_Vertical_I2S_expansion, symbol Connector_Generic:Conn_02x10_Odd_Even
- removed R12: 2.2k ohm - 2200 ohm, project_fp:R_0805_2012Metric_Pad1.20x1.40mm_HandSolder, symbol Device:R
- removed R13, R14, R15: 10k, project_fp:R_0805_2012Metric_Pad1.20x1.40mm_HandSolder, symbol Device:R
- removed S1: PEC12R-2220F-S0024, project_fp:XDCR_PEC12R-2220F-S0024, symbol PEC12R-2220F-S0024:PEC12R-2220F-S0024
- added #EPROG1: header, project_fp:EPROG1_PinHeader_1x06_P2.54mm_Vertical, symbol Connector_Generic:Conn_01x06
- added #SAI2: header, project_fp:IDC-Header_2x10_P2.54mm_Vertical_I2S_expansion, symbol Connector_Generic:Conn_02x10_Odd_Even
- added ESP_I1: header, project_fp:ESP_I2C_0_PinHeader_2x02_P2.54mm_Vertical, symbol Connector_Generic:Conn_02x02_Odd_Even
- added ESP_R_ENC1: header, project_fp:ESP_R_ENC0_PinHeader_1x05_P2.54mm_Vertical, symbol Connector_Generic:Conn_01x05
- added GPI1: header, project_fp:GPI1_PinHeader_1x04_P2.54mm_Vertical, symbol Connector_Generic:Conn_01x04
- added R46, R47, R48, R59, R60: 2.2k ohm - 2200 ohm, project_fp:R_0805_2012Metric_Pad1.20x1.40mm_HandSolder, symbol Device:R
- ILI1, ILI_VCC1: now fitted
Connections:
- net 12V: now also #SAI2.5 (Pin_5)
- net 2_OUT2: now also #SAI2.9 (Pin_9)
- net 3.3V: now also ESP_I1.2 (Pin_2), ESP_R_ENC1.4 (Pin_4), GPI1.3 (Pin_3), R46.1, R47.1, R48.1, R59.1, R60.1
- net 34_RX8_RESET2: now also #SAI2.2 (Pin_2)
- net 35_TX8_RESET: now also #SAI2.1 (Pin_1)
- net 3_LRCLK2: now also #SAI2.13 (Pin_13)
- net 4_BCLK2: now also #SAI2.11 (Pin_11)
- net 5V: now also #SAI2.3 (Pin_3)
- net 5_IN2: now also #SAI2.7 (Pin_7)
- net ESP32_3.3V: now also #EPROG1.4 (Pin_4)
- net ESP32_EN: now also #EPROG1.3 (Pin_3)
- net ESP32_IO0: now also #EPROG1.2 (Pin_2)
- net ESP32_IO1: now also #EPROG1.5 (Pin_5)
- net ESP32_IO3: now also #EPROG1.6 (Pin_6)
- net ESP32_IO33_SPI_CS: now also R48.2
- net GND: now also #EPROG1.1 (Pin_1), #SAI2.10 (Pin_10), #SAI2.12 (Pin_12), #SAI2.14 (Pin_14), #SAI2.16 (Pin_16), #SAI2.18 (Pin_18), #SAI2.20 (Pin_20), #SAI2.4 (Pin_4), #SAI2.6 (Pin_6), #SAI2.8 (Pin_8), ESP_I1.4 (Pin_4), ESP_R_ENC1.5 (Pin_5), GPI1.4 (Pin_4)
- net MCLK2: now also #SAI2.19 (Pin_19)
- net OUTPUTA: now also ESP_R_ENC1.1 (Pin_1)
- net OUTPUTB: now also ESP_R_ENC1.2 (Pin_2)
- net SCL0: now also #SAI2.17 (Pin_17)
- net SDA0: now also #SAI2.15 (Pin_15)
- net SWITCH: now also ESP_R_ENC1.3 (Pin_3)
- net at ILI1.3 (CS), U2.23 (*MTDO/GPIO15/ADC2_CH3): now also R59.2
- net ESP32_IO21_SDA: now reaches U2.33 (GPIO21)
- net ESP32_IO21_SDA: now also ESP_I1.1 (Pin_1), R47.2
- net ESP32_IO22_SCL: now reaches U2.36 (GPIO22)
- net ESP32_IO22_SCL: now also ESP_I1.3 (Pin_3), R46.2
- net at U2.5 (VDET_1/GPIO34/ADC1_CH6): now also GPI1.2 (Pin_2)
- net at U2.6 (VDET_2/GPIO35/ADC1_CH7): now also GPI1.1 (Pin_1)
- net at ILI1.13 (T_CS), U2.7 (32K_XP/GPIO32/ADC1_CH4): now also R60.2
- new net: MIC1.4 (LRCLK-WS-FS), MIC2.4 (LRCLK-WS-FS), board_outline1.40 (GPIO1)
- now unconnected: MIC1.4 (LRCLK-WS-FS), MIC2.4 (LRCLK-WS-FS)
Other:
- moved on the sheet: C31, C32, SW7, SW8, U2

Commit message: update
Parts:
- removed Brd1: SSD1306, project_fp:Adafruit_SSD1306_I2C_ONLY, symbol SSD1306-128x64_OLED:SSD1306
- removed D10, D11, D12, D13, D14, D15, D16, D17, D18, D19, D20, D21, D22, D3, D6, D7, D8, D9: SK6812, project_fp:LED_SK6812_EC15_1.5x1.5mm, symbol SK6812_4020_SIDE_LED:SK6812_REVERSE_MOUNT
- removed D4: HEADER, project_fp:PinHeader_1x04_P2.54mm_Vertical, symbol Connector_Generic:Conn_01x04
- removed IC2: SN74LVC245ARGYR, SN74LVC541ARGYR, symbol SamacSys_Parts:SN74LVC245ARGYR
- removed J2: NMJ6HFD2-AU, Connector_Audio:Jack_6.35mm_Neutrik_NMJ6HFD2-AU_Horizontal, symbol Connector_Audio:NMJ6HFD2-AU
- removed R32, R33, R34: 49.9 ohm, project_fp:R_0805_2012Metric_Pad1.20x1.40mm_HandSolder, symbol Device:R
- removed TDM1, TDM2: header, project_fp:T-DSP_Expansion_Header_2x10_ALT_GND, symbol project_lil_2:TDM_HEADER_Conn_02x10_Odd_Even
- removed U3: TFT_320x240, project_fp:TFT-320x240, symbol tft_320x240:TFT_320x240
- removed U4: EN11-HSM1AF15, project_fp:EN11-HSM_TTE, symbol EN11_HSM1AF15:EN11-HSM1AF15
- added R12, R13: 0 ohm, project_fp:R_0805_2012Metric_Pad1.20x1.40mm_HandSolder, symbol Device:R
- added T_PROG2: header, project_fp:E_PROG1_PinHeader_1x03_P2.54mm_Vertical, symbol Connector_Generic:Conn_01x03
- added U15, U16: Single Buffer - 74LVC1G125GV,125 - SOT-23-5/SC-74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, Package_TO_SOT_SMD:SOT-23-5, symbol project_lil_2:SN74LVC1G125
- C1, C26, C27, C28, C3: now fitted
- D2, D5: footprint project_fp:LED_SK6812_EC15_1.5x1.5mm -> project_fp:LED_4691; now fitted
- SW5, SW6, SW7, SW8: now not fitted
- T_PROG1: now fitted; now in the parts list
Connections:
- net 5V: now also D1.4 (Pin_4), U15.5 (VCC), U16.5 (VCC); no longer D1.2 (Pin_2)
- net ESP32_EN: now also T_PROG2.1 (Pin_1)
- net ESP32_IO0: now also T_PROG2.3 (Pin_3)
- net ESP32_LED: now also U15.2 (A); no longer U2.29 (*GPIO5)
- net GND: now also T_PROG2.2 (Pin_2), U15.1 (OE), U15.3 (GND), U16.1 (OE), U16.3 (GND)
- net TEENSY_LED: now also R11.1, U16.2 (A); no longer R11.2, U1.33 (41_A17)
- net ESP32_LED+: now reaches D2.2 (DOUT)
- net ESP32_LED+: now also D1.1 (Pin_1)
- net at D5.4 (DIN): now also R13.1; no longer R11.1
- net TEENSY_LED+: now reaches D5.2 (DOUT)
- net TEENSY_LED+: now also D1.2 (Pin_2)
- new net: R12.2, U15.4 (Y)
- new net: R7.1, U2.29 (*GPIO5)
- new net: MIC1.4 (LRCLK-WS-FS), MIC2.4 (LRCLK-WS-FS), board_outline1.40 (GPIO1)
- new net: D2.4 (DIN), R12.1
- new net: R11.2, U1.33 (41_A17)
- new net: R13.2, U16.4 (Y)
- now unconnected: MIC1.4 (LRCLK-WS-FS), MIC2.4 (LRCLK-WS-FS)
Other:
- note added: "AUDIO MODULE"
- note added: "CHECK PINS ON LED!!!"
- note added: "HAT MOUNTING POINTS"
- note added: "POWER LED"
- note added: "RGB LED"
- note added: "T-DSP Desktop Soundcard"
- note removed: "STATUS LED"
- note removed: "T-DSP"
- moved on the sheet: 1/4-PHONE1, BAT1, C11, C16, C17, C18, C19, C2, C20, C21, C22, C23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

Commit message: update
Parts:
- removed J3: RCA-IN, project_fp:PJRAS2X1_NOT-VERIFIED, symbol Connector:Conn_Coaxial_x2
- removed J6: RCA-OUT, project_fp:PJRAS2X1_NOT-VERIFIED, symbol Connector:Conn_Coaxial_x2
- added J1, J2: PJRAS2X1S01X, project_fp:PJRAS2X1S01X, symbol PJRAS2X1S01X:PJRAS2X1S01X
- renumbered T_PROG2 to ESP_PROG1
Connections:
- net GND: now also J1.S1, J1.S2, J2.S1, J2.S2
- net IN2_JACK_DETECT: now also J1.T2
- net at HPTRS4.3: now also J1.T1
- net at HPTRS1.3: now also J2.T2
- net at HPTRS1.4: now also J2.T1
- new net: MIC1.4 (LRCLK-WS-FS), MIC2.4 (LRCLK-WS-FS), board_outline1.40 (GPIO1)
- now unconnected: MIC1.4 (LRCLK-WS-FS), MIC2.4 (LRCLK-WS-FS)

Commit message: update
Parts:
- D1: footprint project_fp:PinHeader_1x04_P2.54mm_Vertical -> project_fp:LED_GPIO_PinHeader_1x04_P2.54mm_Vertical
- J1, J2: footprint project_fp:PJRAS2X1S01X -> project_fp:PJRAS2X1S01X_MOD2
Connections:
- new net: MIC1.4 (LRCLK-WS-FS), MIC2.4 (LRCLK-WS-FS), board_outline1.40 (GPIO1)
- now unconnected: MIC1.4 (LRCLK-WS-FS), MIC2.4 (LRCLK-WS-FS)
Changed lines of the file:
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@@
 		(exclude_from_sim no)
 		(in_bom no)
-		(on_board yes)
+		(on_board no)
 		(dnp no)
 		(fields_autoplaced yes)
@@
 			)
 		)
-		(property "Footprint" "project_fp:PJRAS2X1S01X"
+		(property "Footprint" "project_fp:PJRAS2X1S01X_MOD2"
 			(at 547.3692 676.91 0)
 			(effects
@@
 		(exclude_from_sim no)
 		(in_bom no)
-		(on_board yes)
+		(on_board no)
 		(dnp no)
 		(fields_autoplaced yes)
@@
 			)
 		)
-		(property "Footprint" "project_fp:PJRAS2X1S01X"
+		(property "Footprint" "project_fp:PJRAS2X1S01X_MOD2"
 			(at 524.5092 586.74 0)
 			(effects
@@
 			)
 		)
-		(property "Footprint" "project_fp:PJRAS2X1S01X"
+		(property "Footprint" "project_fp:PJRAS2X1S01X_MOD2"
 			(at 547.37 662.94 0)
 			(effects
@@
 			)
 		)
-		(property "Footprint" "project_fp:PJRAS2X1S01X"
+		(property "Footprint" "project_fp:PJRAS2X1S01X_MOD2"
 			(at 524.51 572.77 0)
 			(effects
@@
 		(exclude_from_sim no)
 		(in_bom no)
-		(on_board yes)
+		(on_board no)
 		(dnp no)
 		(fields_autoplaced yes)
@@
 			)
 		)
-		(property "Footprint" "project_fp:PinHeader_1x04_P2.54mm_Vertical"
+		(property "Footprint" "project_fp:LED_GPIO_PinHeader_1x04_P2.54mm_Vertical"
 			(at 1007.11 383.54 0)
 			(effects
@@
 		(exclude_from_sim no)
 		(in_bom no)
-		(on_board yes)
+		(on_board no)
 		(dnp no)
 		(fields_autoplaced yes)

Commit message: update
Parts:
- removed J4: Conn_01x08, Connector_PinHeader_2.54mm:PinHeader_1x08_P2.54mm_Vertical, symbol Connector_Generic:Conn_01x08
- removed USB_IN1: header, project_fp:USB_IN1, symbol project_lil_2:USB_header_1x5_2.54
- added C4: 0.1uF, project_fp:C_0805_2012Metric_Pad1.15x1.40mm_HandSolder, symbol Device:C_Small
- added D3: HEADER, Connector_PinHeader_2.54mm:PinHeader_2x02_P2.54mm_Vertical, symbol Connector_Generic:Conn_01x04
- added R14, R15, R32, R33, R34, R36, R37: 49.9 ohm, project_fp:R_0805_2012Metric_Pad1.20x1.40mm_HandSolder, symbol Device:R
- added U3: SN74LVC245APW, Package_SO:TSSOP-20_4.4x6.5mm_P0.65mm, symbol Logic_LevelTranslator:SN74LVC245APW
- C16, C17, C18, C19, C2, C20, C26, C27, C28, C5, IN1, MIC1, MIC2, OUTA1, OUTC1, R16, R17, R18, R20, R30, R31, R35, U10, U11, U12, U14, U7, U8, U9: now not fitted
- OUTB1, R19, U13: now not fitted; now left out of the parts list
- OUTD1: footprint project_fp:SolderJumper-3_P_23_BRIDGED -> project_fp:SolderJumper-3_P_12_BRIDGED; symbol project_lil_2:SolderJumper_3_Bridged23 -> Jumper:SolderJumper_3_Bridged12; now not fitted; now left out of the parts list
- U1: footprint project_fp:Teensy41_mod -> project_fp:Teensy41_mod3
- renumbered TDM3 to TDM1, TDM4 to TDM2
Connections:
- net 3.3V: now also C4.1, U3.20 (VCC)
- net 5V: now also RLED1.2, USBC1.A4 (VBUS), USBC1.A9 (VBUS), USBC1.B4 (VBUS), USBC1.B9 (VBUS)
- net 5VIN2: no longer USBC1.A4 (VBUS), USBC1.A9 (VBUS), USBC1.B4 (VBUS), USBC1.B9 (VBUS)
- net 6_OUT1D: now also U3.4 (A3)
- net 6_OUT1D+: now also TDM2.7 (DSP_DATA_IN), R37.2
- net 7_OUT1A: now also U3.17 (B2)
- net 7_OUT1A+: now also R33.2; no longer TDM2.9 (DSP_DATA_OUT)
- net 8_IN1: now also U3.2 (A1)
- net 8_IN1+: now also R36.2; no longer TDM2.7 (DSP_DATA_IN)
- net 9_OUT1C: now also U3.15 (B4)
- net 9_OUT1C+: now also TDM2.9 (DSP_DATA_OUT), R34.2
- net BCLK1: now also U3.13 (B6)
- net BCLK1+: now also R15.2
- net GND: now also PWR1.1 (K), C4.2, U3.12 (B7), U3.8 (A7)
- net LRCK1: now also U3.14 (B5)
- net LRCK1+: now also R14.2
- net MCLK1: now also U3.11 (B8)
- net MCLK1+: now also R32.2
- net MIDI_RX: now also U1.2 (0_RX1_CRX2_CS1)
- net MIDI_TX_T: now also U1.3 (1_TX1_CTX2_MISO1)
- net at board_outline1.41 (GPIO2): now also D3.2 (Pin_2)
- net at board_outline1.42 (GPO1): now also D3.3 (Pin_3)
- net at MIC1.1 (DATA), MIC2.1 (DATA), board_outline1.43 (GPI1): now also D3.4 (Pin_4)
- new net: R15.1, U3.7 (A6)
- new net: R34.1, U3.5 (A4)
- new net: D3.1 (Pin_1), MIC1.4 (LRCLK-WS-FS), MIC2.4 (LRCLK-WS-FS), board_outline1.40 (GPIO1)
- new net: R33.1, U3.3 (A2)
- new net: R37.1, U3.16 (B3)
- new net: R36.1, U3.18 (B1)
- new net: R14.1, U3.6 (A5)
- new net: R32.1, U3.9 (A8)
- now unconnected: MIC1.4 (LRCLK-WS-FS), MIC2.4 (LRCLK-WS-FS)
- no-connect marks 12 -> 13
Other:
- note added: "USB IN HEADER"
- note removed: "5VIN to Current Limiter/Switch"
- note removed: "Post Current Limiter/Switch"
- moved on the sheet: PWR1, RLED1, TDM1, TDM2

Commit message: update
Parts:
- added JP1, JP2: Jumper_2_Open, project_fp:jumper_slice_disconnected, symbol Jumper:Jumper_2_Open
- D2, D5: footprint project_fp:LED_4691 -> project_fp:SK6812-32228SMD-Reverse-Mount; symbol SK6812_4020_SIDE_LED:SK6812_REVERSE_MOUNT -> LED_4691_SK6812_SIDE_MOUNT:LED_4691_SK6812_SIDE_MOUNT
Connections:
- net 5V: now also D2.2 (VDD), D5.2 (VDD); no longer D2.1 (VDD), D5.1 (VDD)
- net ESP32_LED+: now also D2.3 (DOUT), JP2.2 (B); no longer D2.2 (DOUT)
- net GND: now also D2.4 (GND), D5.4 (GND); no longer D2.3 (GND), D5.3 (GND)
- net TEENSY_LED+: now also D5.3 (DOUT), JP1.2 (B); no longer D5.2 (DOUT)
- net at R12.1: now also D2.1 (DIN), JP2.1 (A); no longer D2.4 (DIN)
- net at R13.1: now also D5.1 (DIN), JP1.1 (A); no longer D5.4 (DIN)
Other:
- moved on the sheet: C1, D5, R13, U16
