File: audio_back_plane_35_rca.kicad_sch (KiCad schematic)
At the start: 148 parts, among them IC3 TMUX4052BQBR, IC5 TMUX4053DYYR, J1 PJRAS2X1S01X, J2 PJRAS2X1S01X, SW1 RotaryEncoder_Switch_MP, SW2 TL1105WF160Q - 3.15mm actuator, SW3 TL1105WF160Q - 3.15mm actuator, SW4 TL1105WF160Q - 3.15mm actuator, SW5 SW_SPST, SW6 TL1105WF160Q - 3.15mm actuator, SW7 SW_SPST, SW8 SW_SPST, U1 Teensy 4.1 - DEVKIT, U10 SN74LVC1T45DBV, U11 SN74LVC1T45DBV, U12 SN74LVC1T45DBV, U13 SN74LVC1T45DBV, U14 Single Buffer - 74LVC1G125GV,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, U15 Single Buffer - 74LVC1G125GV,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, U16 Single Buffer - 74LVC1G125GV,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, U2 ESP32-DevKitC - DEVKIT, U3 SN74LVC245APW, U5 Optoisolators - H11L1SM - 6-S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, U6 Dual Buffer - 74HCT2G17GW,125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, U7 Single Buffer - 74LVC1G125GV,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, U8 Single Buffer - 74LVC1G125GV,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, U9 SN74LVC1T45DBV

Commit message: update
Parts:
- added R38, R39: 49.9 ohm, project_fp:R_0805_2012Metric_Pad1.20x1.40mm_HandSolder, symbol Device:R
- D3: footprint Connector_PinHeader_2.54mm:PinHeader_2x02_P2.54mm_Vertical -> project_fp:TAC5212_GPIO_PinHeader_2x02_P2.54mm_Vertical
Connections:
- net 6_OUT1D: now also U3.8 (A7), R38.2; no longer U1.8 (6_OUT1D), U3.4 (A3)
- net 7_OUT1A: now also U3.13 (B6), R39.2; no longer U1.9 (7_RX2_OUT1A), U3.17 (B2)
- net 8_IN1: now also U3.6 (A5); no longer U3.2 (A1)
- net 9_OUT1C: now also U3.11 (B8); no longer U3.15 (B4)
- net BCLK1: now also U3.16 (B3); no longer U3.13 (B6)
- net BCLK1+: now also R14.2; no longer R15.2
- net GND: now also U3.10 (GND), U3.17 (B2), U3.3 (A2); no longer U3.12 (B7), U3.8 (A7)
- net LRCK1: now also U3.15 (B4); no longer U3.14 (B5)
- net LRCK1+: now also R15.2; no longer R14.2
- net MCLK1: now also U3.18 (B1); no longer U3.11 (B8)
- net at R15.1: now also U3.5 (A4); no longer U3.7 (A6)
- net at R34.1: now also U3.9 (A8); no longer U3.5 (A4)
- net at R33.1: now also U3.7 (A6); no longer U3.3 (A2)
- net at R37.1: now also U3.12 (B7); no longer U3.16 (B3)
- net at R36.1: now also U3.14 (B5); no longer U3.18 (B1)
- net at R14.1: now also U3.4 (A3); no longer U3.6 (A5)
- net at R32.1: now also U3.2 (A1); no longer U3.9 (A8)
- new net: R38.1, U1.8 (6_OUT1D)
- new net: R39.1, U1.9 (7_RX2_OUT1A)
Other:
- moved on the sheet: R14, R15, R32, R33, R34, R36, R37

Commit message: Update audio_back_plane_35_rca.kicad_sch
Parts:
- removed R6: 10k, project_fp:R_0805_2012Metric_Pad1.20x1.40mm_HandSolder, symbol Device:R
Connections:
- net SCL_C is gone; now on net SCL0: TDM2.17 (SCL)
- net SCL_D is gone; now on net SCL0: TDM1.17 (SCL)
- net SDA_C is gone; now on net SDA0: TDM2.15 (SDA)
- net SDA_D is gone; now on net SDA0: TDM1.15 (SDA)
- net 34_RX8_RESET2: now also U1.26 (34_RX8)
- net GND: no longer J1.S1
- net IN2_JACK_DETECT: no longer HPTRS4.4, J1.T2
- net at HPTRS4.3: no longer J1.T1
- new net: HPTRS4.4, J1.T2
Other:
- note added: "B) High-speed first, analog last (when fast buses are critical) L1: High-speed signals and clocks L2: Solid GND L3: High-speed or dense digital fanout L4: Power L5: Solid GND L6: Analog signals and sensitive I/O"
- moved on the sheet: J1A

Commit message: update
Connections:
- net GND: now also J1.T1
- net at HPTRS4.3: now also J1.S1
Other:
- moved on the sheet: J1A
Changed lines of the file:
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@@
 	(symbol
 		(lib_id "PJRAS2X1S01X:PJRAS2X1S01X")
-		(at 547.37 662.94 0)
+		(at 547.37 662.94 180)
 		(unit 1)
 		(exclude_from_sim no)
@@
 		(dnp no)
 		(property "Reference" "J1"
-			(at 547.3655 655.32 0)
+			(at 547.3745 670.56 0)
 			(effects
 				(font
@@
 		)
 		(property "Value" "PJRAS2X1S01X"
-			(at 547.3655 657.86 0)
+			(at 547.3745 668.02 0)
 			(effects
 				(font

Commit message: update
Parts:
- removed C1, C3: 0.1uF, project_fp:C_0805_2012Metric_Pad1.15x1.40mm_HandSolder, symbol TEENSY_4.0_ESP32_AUDIO-rescue:C_Small-Device
- removed C17, C18, C23, C24, C25, C26, C27, C28, C29, C30: 0.1uF, project_fp:C_0805_2012Metric_Pad1.15x1.40mm_HandSolder, symbol Device:C_Small
- removed JP1, JP2: Jumper_2_Open, project_fp:jumper_slice_disconnected, symbol Jumper:Jumper_2_Open
- removed R12, R13: 0 ohm, project_fp:R_0805_2012Metric_Pad1.20x1.40mm_HandSolder, symbol Device:R
- removed U15, U16: Single Buffer - 74LVC1G125GV,125 - SOT-23-5/SC-74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, Package_TO_SOT_SMD:SOT-23-5, symbol project_lil_2:SN74LVC1G125
- added C1, C10, C12, C13, C14, C15, C3, C6, C9: 0.1uF, project_fp:C_0805_2012Metric_Pad1.15x1.40mm_HandSolder, symbol Device:C_Small
- added C17: 0.1uF, project_fp:C_0805_2012Metric_Pad1.15x1.40mm_HandSolder, symbol TEENSY_4.0_ESP32_AUDIO-rescue:C_Small-Device
- added C18: 10uF, project_fp:C_0805_2012Metric_Pad1.15x1.40mm_HandSolder, symbol TEENSY_4.0_ESP32_AUDIO-rescue:C_Small-Device
- added IC1: 74HCT2G125DC,125, project_fp:SOP50P310X100-8N, symbol 74HCT2G125DC_125:74HCT2G125DC,125
- added R41, R42, R43, R6: 33Ω, project_fp:R_0805_2012Metric_Pad1.20x1.40mm_HandSolder, symbol Device:R
- added U17, U18, U19, U20, U4: Single Buffer - 74LVC1G125GV,125 - SOT-23-5/SC-74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, Package_TO_SOT_SMD:SOT-23-5, symbol project_lil_2:SN74LVC1G125
- added U21, U22, U23, U24: SN74LVC2G125DCTR, project_fp:SOP65P400X130-8N, symbol SN74LVC2G125DCTR:SN74LVC2G125DCTR
- C19, C20: now fitted
- C4, R14, R15, R32, R33, R34, R36, R37, U3: now not fitted; now left out of the parts list
- D2, D5: footprint project_fp:SK6812-32228SMD-Reverse-Mount -> project_fp:SK6812-32228SMD-Reverse-Mount_mod
- R20, R30, R31: value 0 ohm -> 33Ω
- R40: value 0ohm -> 33Ω; 2020-10-01 PARTS RPC0805JT100K -> (none); Package / Case (none) -> R0805; mouser (none) -> 603-RC0805DR-072K2L
Connections:
- net 3.3V: now also C16.1, C19.1, C20.1, U14.5 (VCC), U7.5 (VCC), U8.5 (VCC), C1.1, C10.1, C12.1, C13.1, C14.1, C15.1, C3.1, C6.1, C9.1, U17.5 (VCC), U18.5 (VCC), U19.5 (VCC), U20.5 (VCC), U21.8 (VCC), U22.8 (VCC), U23.8 (VCC), U24.8 (VCC), U4.5 (VCC); no longer R40.2
- net 3.3V_BUFFER: no longer C16.1, C19.1, C20.1, R40.1, U14.5 (VCC), U7.5 (VCC), U8.5 (VCC)
- net 32_OUT1B: now also U20.2 (A)
- net 32_OUT1B+: now also R43.1
- net 5V: now also C17.1, C18.1, IC1.8 (VCC); no longer D1.4 (Pin_4)
- net 6_OUT1D: now also U24.5 (2A); no longer U3.8 (A7)
- net 6_OUT1D+: now also TDM2.9 (DSP_DATA_OUT), U24.3 (2Y); no longer R37.2, TDM2.7 (DSP_DATA_IN)
- net 7_OUT1A: now also U19.2 (A), U24.2 (1A); no longer board_outline1.7 (DSP_DOUT)
- net 7_OUT1A+: now also board_outline1.7 (DSP_DOUT), R42.1, U24.6 (1Y)
- net 8_IN1: now also TDM1.7 (DSP_DATA_IN)
- net 8_IN1+: no longer TDM1.7 (DSP_DATA_IN)
- net 9_OUT1C: no longer U1.11 (9_OUT1C)
- net 9_OUT1C+: no longer TDM2.9 (DSP_DATA_OUT)
- net BCLK1: now also U18.2 (A), U23.2 (1A), U23.5 (2A); no longer board_outline1.11 (BCLK)
- net BCLK1+: no longer R31.1, TDM1.11 (BCLK), TDM2.11 (BCLK)
- net ESP32_LED: now also IC1.2 (1A)
- net ESP32_LED+: now also D2.1 (DIN), IC1.6 (1Y); no longer D1.1 (Pin_1), D2.3 (DOUT)
- net GND: now also C1.2, C10.2, C12.2, C13.2, C14.2, C15.2, C17.2, C18.2, C3.2, C6.2, C9.2, IC1.1 (~{1OE}), IC1.4 (GND), IC1.7 (~{2OE}), U17.1 (OE), U17.3 (GND), U18.1 (OE), U18.3 (GND), U19.1 (OE), U19.3 (GND), U20.1 (OE), U20.3 (GND), U21.1 (~{1OE}), U21.4 (GND), U21.7 (~{2OE}), U22.1 (~{1OE}), U22.4 (GND), U22.7 (~{2OE}), U23.1 (~{1OE}), U23.7 (~{2OE}), U4.1 (OE), U4.3 (GND)
- net LRCK1: now also U17.2 (A), U22.2 (1A), U22.5 (2A); no longer board_outline1.13 (LRCK)
- net LRCK1+: no longer R30.1, TDM1.13 (LRCK), TDM2.13 (LRCK)
- net MCLK1: now also U21.2 (1A), U21.5 (2A), U4.2 (A); no longer board_outline1.19 (MCLK)
- net MCLK1+: no longer R20.1, TDM1.19 (MCLK), TDM2.19 (MCLK)
- net TEENSY_LED: now also IC1.5 (2A)
- net TEENSY_LED+: now also D5.1 (DIN), IC1.3 (2Y); no longer D1.2 (Pin_2), D5.3 (DOUT)
- new net: R40.2, U17.4 (Y)
- new net: R6.2, U4.4 (Y)
- new net: R43.2, U20.4 (Y)
- new net: R42.2, U19.4 (Y)
- new net: R41.2, U18.4 (Y)
- new net 9_OUT1C_INPUT: TDM2.7 (DSP_DATA_IN), U1.11 (9_OUT1C)
- new net BCLK1+TDM1: R31.1, TDM1.11 (BCLK), U23.6 (1Y), board_outline1.11 (BCLK)
- new net BCLK1+TDM2: R41.1, TDM2.11 (BCLK), U23.3 (2Y)
- new net ESP32_LED_OUT: D1.1 (Pin_1), D2.3 (DOUT)
- new net LED_PWR: D1.4 (Pin_4)
- new net LRCK1+TDM1: R30.1, TDM1.13 (LRCK), U22.6 (1Y), board_outline1.13 (LRCK)
- new net LRCK1+TDM2: R40.1, TDM2.13 (LRCK), U22.3 (2Y)
- new net MCLK1+TDM1: R20.1, TDM1.19 (MCLK), U21.6 (1Y), board_outline1.19 (MCLK)
- new net MCLK1+TDM2: R6.1, TDM2.19 (MCLK), U21.3 (2Y)
- new net TEENSY_LED_OUT: D1.2 (Pin_2), D5.3 (DOUT)
Other:
- note added: "CLOCK DRIVER TDM1"
- note added: "CLOCK DRIVER TDM2"
- note removed: "CHECK PINS ON LED!!!"
- note removed: "CLOCK DRIVER"
- moved on the sheet: D1, D2, D5, IN1, OUTA1, OUTB1, OUTC1, OUTD1, R16, R17, R18, R19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

Commit message: update
Other:
- note added: "KiCad 8-Layer Stackup: F.Cu - TOP: Components, ANALOG routes to jacks, ground fill In1.Cu - GND: Solid ground plane In2.Cu - SIG1: TDM/high-speed digital, ground fill In3.Cu - GND: Solid ground plane (isolation!) In4.Cu - SIG2: More TDM/digital signals, ground fill In5.Cu - PWR: Power planes (3.3V/5V) In6.Cu - GND: Solid ground plane B.Cu - BOTTOM: Components, ANALOG routes to jacks, ground fill"
- note removed: "B) High-speed first, analog last (when fast buses are critical) L1: High-speed signals and clocks L2: Solid GND L3: High-speed or dense digital fanout L4: Power L5: Solid GND L6: Analog signals and sensitive I/O"
Changed lines of the file:
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@@
 		)
 	)
-	(text "B) High-speed first, analog last (when fast buses are critical)\n\nL1: High-speed signals and clocks\n\nL2: Solid GND\n\nL3: High-speed or dense digital fanout\n\nL4: Power\n\nL5: Solid GND\n\nL6: Analog signals and sensitive I/O"
+	(text "KiCad 8-Layer Stackup:\nF.Cu    - TOP: Components, ANALOG routes to jacks, ground fill\nIn1.Cu  - GND: Solid ground plane\nIn2.Cu  - SIG1: TDM/high-speed digital, ground fill\nIn3.Cu  - GND: Solid ground plane (isolation!)\nIn4.Cu  - SIG2: More TDM/digital signals, ground fill\nIn5.Cu  - PWR: Power planes (3.3V/5V)\nIn6.Cu  - GND: Solid ground plane\nB.Cu    - BOTTOM: Components, ANALOG routes to jacks, ground fill"
 		(exclude_from_sim no)
 		(at -372.872 299.72 0)

Commit message: update
Parts:
- added BAT2: BAT, project_fp:BAT2_PinSocket_1x02_P2.54mm_Vertical, symbol Connector_Generic:Conn_01x02
- added INPUT1, OUT1: Conn_02x02_Odd_Even, Connector_PinHeader_2.54mm:PinHeader_2x02_P2.54mm_Vertical, symbol Connector_Generic:Conn_02x02_Odd_Even
- added J3: Conn_01x01_Pin, project_fp:GPIO_GROUND_PinHeader_1x01_P2.54mm_Vertical, symbol Connector:Conn_01x01_Pin
- added J4, J5, J6, J7, J8, J9: jumper, project_fp:jumper_slice_disconnected, symbol JUMPER:JUMPER_SMALL
- D3: footprint project_fp:TAC5212_GPIO_PinHeader_2x02_P2.54mm_Vertical -> project_fp:TAC5212 GPIO_PinHeader_1x06_P2.54mm_Vertical; symbol Connector_Generic:Conn_01x04 -> Connector_Generic:Conn_01x06
- ESP_I1: footprint project_fp:ESP_I2C_0_PinHeader_2x02_P2.54mm_Vertical -> project_fp:ESP_I2C_PinHeader_1x04_P2.54mm_Vertical
Connections:
- net SYSTEM_EN is gone; now on net 3.3V: TDM1.4 (GND), TDM2.4 (GND)
- net 3.3V: now also D3.5 (Pin_5), board_outline1.4 (GNDD)
- net 34_RX8_RESET2: now also board_outline1.2 (HELD_LOW)
- net GND: now also D3.6 (Pin_6), INPUT1.2 (Pin_2), INPUT1.4 (Pin_4), OUT1.2 (Pin_2), OUT1.4 (Pin_4); no longer board_outline1.4 (GNDD)
- net at 1/4-PHONE1.R, board_outline1.21 (OUTP): now also J7.1, OUT1.1 (Pin_1)
- net at 1/4-PHONE1.RN, HPTRS1.2: now also J7.2, J9.1
- net at 1/4-PHONE1.T, board_outline1.25 (OUT2P): now also J6.2, OUT1.3 (Pin_3)
- net at 1/4-PHONE1.TN, HPTRS1.5: now also J6.1, J8.2
- net at BAT1.1 (+), U1.50 (VBAT): now also BAT2.1 (Pin_1)
- net at BAT1.2 (-), U1.52 (GND): now also BAT2.2 (Pin_2)
- net at HPTRS4.2, board_outline1.29 (IN1P): now also INPUT1.3 (Pin_3), J5.1
- net at HPTRS4.3, J1.S1: now also J5.2
- net at HPTRS4.4, J1.T2: now also J4.1
- net at HPTRS4.5, board_outline1.33 (IN2P): now also INPUT1.1 (Pin_1), J4.2
- net at HPTRS1.3, J2.T2: now also J9.2
- net at HPTRS1.4, J2.T1: now also J8.1
Other:
- moved on the sheet: HPTRS4, J1A, J1B, T_PROG1

Commit message: update
Connections:
- net GND: now also J1.S1; no longer J1.T1
- net at HPTRS4.3, J5.2: now also J1.T1; no longer J1.S1
Other:
- moved on the sheet: J1A
Changed lines of the file:
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@@
 	(symbol
 		(lib_id "PJRAS2X1S01X:PJRAS2X1S01X")
-		(at 566.42 662.94 180)
+		(at 566.42 662.94 0)
+		(mirror y)
 		(unit 1)
 		(exclude_from_sim no)
@@
 		(dnp no)
 		(property "Reference" "J1"
-			(at 566.4245 670.56 0)
+			(at 566.4245 655.32 0)
 			(effects
 				(font
@@
 		)
 		(property "Value" "PJRAS2X1S01X"
-			(at 566.4245 668.02 0)
+			(at 566.4245 657.86 0)
 			(effects
 				(font

Commit message: update
Connections:
- no-connect marks 13 -> 15
Changed lines of the file:
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@@
+	)
+	(no_connect
+		(at 1070.61 568.96)
+	)
+	(no_connect
+		(at 1070.61 571.5)
 	)
 	(no_connect
