File: t-dsp_desktop_pro.kicad_sch (KiCad schematic)
At the start: 174 parts, among them IC1 Logic Level Shifter - 74HCT2G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, J1 jumper, J10 JST-XH Connector -, J11 JST-XH Connector -, J12 RGB LED HEADEER, J13 Conn_02x02_Odd_Even, J14 Conn_01x03, J15 Conn_01x01, J2 GROUND HEADER, J3 jumper, J4 jumper, J5 jumper, J6 jumper, J7 jumper, J8 PJRAS2X1S01X, J9 PJRAS2X1S01X, SW1 SW_SPST, SW2 TL1105WF160Q - 3.15mm actuator, SW3 SW_SPST, SW4 SW_SPST, SW5 RotaryEncoder_Switch_MP, SW6 TL1105WF160Q - 3.15mm actuator, SW7 TL1105WF160Q - 3.15mm actuator, SW8 TL1105WF160Q - 3.15mm actuator, T108 Tab, T109 Tab, T110 Tab, T111 Tab, U1 Teensy 4.1 - DEVKIT, U2 ESP32-DevKitC - DEVKIT, U3 Power Mux & Protect - TPS2116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, U4 Optoisolators - H11L1SM - 6-S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, U5 Dual Buffer - SN74LVC2G125DCTR, U6 Dual Buffer - SN74LVC2G125DCTR, U7 Dual Buffer - SN74LVC2G125DCTR, U8 Dual Buffer - SN74LVC2G125DCTR, U9 Dual Buffer - 74HCT2G17GW,125

Commit message: Add KiBot CI pipeline, bundle 3D models locally, fix Blender renders
- Add .kibot.yaml with full manufacturing outputs (gerbers, BOM, 3D renders)
- Add GitHub Actions workflow for automated manufacturing file generation
- Bundle ~26 standard KiCad library 3D models into 3d_models/ so they
  resolve in Docker/CI without a KiCad installation
- Rewrite all PCB model paths from ${KISYS3DMOD}/${KICAD*_3DMODEL_DIR}
  to ${KIPRJMOD}/3d_models/ for portable resolution
- Fix broken model refs (hardcoded Windows path, bare filename)
- Set kicad_dnp_applies_to_3D: false so DNP-flagged schematic symbols
  (used for BOM filtering) keep their 3D models in Blender renders
- Add local Docker test script (scripts/test_3d_local.sh)

Co-Authored-By: Claude Opus 4.6 <noreply@anthropic.com>
Parts:
- added J17: Conn_02x04_Odd_Even, project_fp:PinHeader_2x04_P2.54mm_Vertical_MIDI_IO, symbol Connector_Generic:Conn_02x04_Odd_Even
- added J18: Conn_02x02_Odd_Even, project_fp:PinHeader_2x02_P2.54mm_Vertical_SPDIF_IO, symbol Connector_Generic:Conn_02x02_Odd_Even
- BAT1: footprint project_fp:BAT2_PinSocket_1x02_P2.54mm_Vertical -> Connector_PinHeader_2.54mm:PinHeader_1x02_P2.54mm_Vertical
- SPDIF_IO1: now left out of the parts list
- TDM1, TDM2: value I2S /I2C EXPANSION HEADER -> T-DSP_expansion_header
- renumbered 1/4-PHONE1 to J_PHONE1
Connections:
- net 14_SPDIF_OUT: now also J18.3 (Pin_3)
- net 15_SPDIF_IN: now also J18.1 (Pin_1)
- net 3.3V: now also J18.4 (Pin_4)
- net 5V: now also J18.2 (Pin_2)
- net GND: now also J17.7 (Pin_7), J17.8 (Pin_8)
- net MIDI_IN_4: now also J17.1 (Pin_1)
- net MIDI_IN_5: now also J17.2 (Pin_2)
- net MIDI_OUT_4: now also J17.3 (Pin_3)
- net MIDI_OUT_5: now also J17.4 (Pin_4)
- net MIDI_THRU_4: now also J17.5 (Pin_5)
- net MIDI_THRU_5: now also J17.6 (Pin_6)
