File: t-dsp_desktop_pro.kicad_sch (KiCad schematic)
At the start: 176 parts, among them IC1 Logic Level Shifter - 74HCT2G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, J1 jumper, J10 JST-XH Connector -, J11 JST-XH Connector -, J12 RGB LED HEADEER, J13 Conn_02x02_Odd_Even, J14 Conn_01x03, J15 Conn_01x01, J17 Conn_02x04_Odd_Even, J18 Conn_02x02_Odd_Even, J2 GROUND HEADER, J3 jumper, J4 jumper, J5 jumper, J6 jumper, J7 jumper, J8 PJRAS2X1S01X, J9 PJRAS2X1S01X, SW1 SW_SPST, SW2 TL1105WF160Q - 3.15mm actuator, SW3 SW_SPST, SW4 SW_SPST, SW5 RotaryEncoder_Switch_MP, SW6 TL1105WF160Q - 3.15mm actuator, SW7 TL1105WF160Q - 3.15mm actuator, SW8 TL1105WF160Q - 3.15mm actuator, T108 Tab, T109 Tab, T110 Tab, T111 Tab, U1 Teensy 4.1 - DEVKIT, U2 ESP32-DevKitC - DEVKIT, U3 Power Mux & Protect - TPS2116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, U4 Optoisolators - H11L1SM - 6-S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, U5 Dual Buffer - SN74LVC2G125DCTR, U6 Dual Buffer - SN74LVC2G125DCTR, U7 Dual Buffer - SN74LVC2G125DCTR, U8 Dual Buffer - SN74LVC2G125DCTR, U9 Dual Buffer - 74HCT2G17GW,125

Commit message: update
Parts:
- removed J13: Conn_02x02_Odd_Even, symbol Connector_Generic:Conn_02x02_Odd_Even
- added J13, J16: Conn_01x02, project_fp:PinHeader_1x02_P2.54mm_Vertical_NO_CTYD, symbol Connector_Generic:Conn_01x02
- added J20: t-dsp_desktop_pro, symbol lib_sch:t-dsp_desktop_pro
- BAT2: Package / Case (none) -> BATTERY
- C24, C25, C26: mouser 581-08055C104M4T4A -> (none)
- C6, C8: Package / Case (none) -> 7343-15
- D1, J17, U2: Package / Case (none) -> HEADER
- H1, H2, H3, H4: Package / Case (none) -> HOLE; now not fitted
- ILI_VCC1, J1, J3, J4, J5, J6, J7, MIDI_OT1, MIDI_OT2: now not fitted
- J14, J15, J18: Package / Case (none) -> HEADER; now not fitted
- MIC1, MIC2: Package / Case (none) -> SMD-MIC
- MIDI_OUT_1: Package / Case through-hole -> TH-JACK; now not fitted
- R24: Package / Case (none) -> R0805
- R5, R52: now fitted
- SW1, SW2, SW3, SW4, SW5, SW6, SW7, SW8: Package / Case (none) -> TH-SWITCH
- T108, T109, T110, T111: Package / Case (none) -> TAB; now not fitted
- USBB1: Package / Case (none) -> TH-JACK
Connections:
- net T_BUTTON1: now also J16.1 (Pin_1)
- net T_BUTTON2: now also J16.2 (Pin_2)
- net at J14.2 (Pin_2), R52.2: now also J13.2 (Pin_2)
- net at J14.1 (Pin_1), U1.22 (30_CRX3): now also J13.1 (Pin_1)
- net IN2_JACK_DETECT: no longer names the net of U1.18 (26_A12_MOSI1)

Commit message: created expansion board outline with headers
Parts:
- removed J20: t-dsp_desktop_pro, symbol lib_sch:t-dsp_desktop_pro
- J14: now left out of the parts list
- TDM1: renamed from TDM2; symbol project_lil_2:TDM_HEADER_Conn_02x10_Odd_Even -> lib_sch:TDM_HEADER_Conn_02x10_Odd_Even
- TDM2: renamed from TDM1; symbol project_lil_2:TDM_HEADER_Conn_02x10_Odd_Even -> lib_sch:TDM_HEADER_Conn_02x10_Odd_Even
- board_outline2: symbol project_lil_2:audio_project_board -> lib_sch:t-dsp_desktop_pro; now in the parts list
Connections:
- net 12V: now also board_outline2.T5 (12V), board_outline2.TT5 (Pin_5)
- net 14_SPDIF_OUT: now also board_outline2.11 (OUT)
- net 15_SPDIF_IN: now also board_outline2.9 (IN)
- net 3.3V: now also board_outline2.45 (3.3), board_outline2.T4 (3.3V), board_outline2.TT4 (Pin_4)
- net 34_RX8_RESET2: now also board_outline2.T2 (HELD_LOW), board_outline2.TT2 (Pin_2)
- net 35_TX8_RESET: now also board_outline2.T1 (HELD_HIGH), board_outline2.TT1 (Pin_1)
- net 53_T_PROG: now also board_outline2.55 (?)
- net 54_ON_OFF: now also board_outline2.59 (OFF)
- net 5V: now also board_outline2.T3 (5V), board_outline2.TT3 (Pin_3)
- net 6_OUT1D+: now also board_outline2.TT9 (Pin_9)
- net 7_OUT1A+: now also board_outline2.T9 (DSP_DATA_OUT)
- net 8_IN1: now also board_outline2.T7 (DSP_DATA_IN)
- net 9_OUT1C_INPUT: now also board_outline2.TT7 (Pin_7)
- net BCLK1+TDM1: now also board_outline2.T11 (BCLK)
- net BCLK1+TDM2: now also board_outline2.TT11 (Pin_11)
- net ESP32_IO21_SDA: now also board_outline2.43 (SD)
- net ESP32_IO22_SCL: now also board_outline2.47 (SC)
- net GND: now also BAT1.2 (Pin_2), BAT2.2 (-), J2.1 (Pin_1), U1.52 (GND), board_outline2.13 (G), board_outline2.17 (G), board_outline2.49 (G), board_outline2.57 (G), board_outline2.7 (G), board_outline2.T10 (GND), board_outline2.T12 (GND), board_outline2.T14 (GND), board_outline2.T16 (GND), board_outline2.T18 (GND), board_outline2.T20 (GND), board_outline2.T6 (GND), board_outline2.T8 (GND), board_outline2.TT10 (Pin_10), board_outline2.TT12 (Pin_12), board_outline2.TT14 (Pin_14), board_outline2.TT16 (Pin_16), board_outline2.TT18 (Pin_18), board_outline2.TT20 (Pin_20), board_outline2.TT6 (Pin_6), board_outline2.TT8 (Pin_8)
- net LED: now also ILI1.8 (LED_(3.3V)), R24.2, board_outline2.29 (LED)
- net LRCK1+TDM1: now also board_outline2.T13 (LRCK)
- net LRCK1+TDM2: now also board_outline2.TT13 (Pin_13)
- net MCLK1+TDM1: now also board_outline2.T19 (MCLK)
- net MCLK1+TDM2: now also board_outline2.TT19 (Pin_19)
- net MIDI_IN_4: now also board_outline2.1 (I4)
- net MIDI_OUT_4: now also board_outline2.3 (O4)
- net MIDI_THRU_4: now also board_outline2.5 (T4)
- net SCL0: now also board_outline2.T17 (SCL)
- net SCL1: now also board_outline2.TT17 (Pin_17)
- net SDA0: now also board_outline2.T15 (SDA)
- net SDA1: now also board_outline2.TT15 (Pin_15)
- net V_BAT: now reaches BAT1.1 (Pin_1), BAT2.1 (+), U1.50 (VBAT)
- net V_BAT: now also board_outline2.61 (BAT)
- net TRX3: now reaches J13.2 (Pin_2), J14.2 (Pin_2), R52.2
- net TRX3: now also board_outline2.53 (?)
- net at R50.2: now also board_outline2.B2; no longer board_outline2.3 (GND)
- net CS: now reaches ILI1.3 (CS), R22.2, U2.23 (*MTDO/GPIO15/ADC2_CH3)
- net CS: now also board_outline2.19 (CS)
- net DC: now reaches ILI1.5 (DC), U2.24 (ADC2_CH2/*GPIO2)
- net DC: now also board_outline2.23 (DC)
- net RESET: now reaches ILI1.4 (RESET), U2.26 (ADC2_CH0/GPIO4)
- net RESET: now also board_outline2.21 (RS)
- net SCK: now reaches ILI1.10 (T_CLK(SCK)), ILI1.7 (SCK), U2.30 (GPIO18)
- net SCK: now also board_outline2.27 (SCK), board_outline2.33 (CK)
- net SDO: now reaches ILI1.13 (T_DO(MISO)), ILI1.9 (SDO(MISO)), U2.31 (GPIO19)
- net SDO: now also board_outline2.31 (X), board_outline2.39 (DO)
- net SDI: now reaches ILI1.12 (T_DIN(MOSI)), ILI1.6 (SDI(MOSI)), U2.37 (GPIO23)
- net SDI: now also board_outline2.25 (DI), board_outline2.37 (DI)
- net GPIO34: now reaches GPI1.2 (Pin_2), U2.5 (VDET_1/GPIO34/ADC1_CH6)
- net GPIO35: now reaches GPI1.1 (Pin_1), U2.6 (VDET_2/GPIO35/ADC1_CH7)
- net T_CS: now reaches ILI1.11 (T_CS), R23.2, U2.7 (32K_XP/GPIO32/ADC1_CH4)
- net T_CS: now also board_outline2.35 (CS)
- net CRX3: now reaches J13.1 (Pin_1), J14.1 (Pin_1), U1.22 (30_CRX3)
- net CRX3: now also board_outline2.51 (?)
- net GPIO1: now reaches D1.1 (Pin_1), MIC1.4 (LRCLK-WS-FS), MIC2.4 (LRCLK-WS-FS), board_outline1.40 (GPIO1)
- net GPIO2: now reaches D1.2 (Pin_2), board_outline1.41 (GPIO2)
- net GPO1: now reaches D1.3 (Pin_3), board_outline1.42 (GPO1)
- net GPIGPI1: now reaches D1.4 (Pin_4), MIC1.1 (DATA), MIC2.1 (DATA), board_outline1.43 (GPI1)
- net VCC: now reaches ILI1.1 (VCC_(5V)), ILI_VCC1.2 (C)
- net VCC: now also board_outline2.15 (VCC)
- net IRQ: now reaches ILI1.14 (T_IRQ)
- net IRQ: now also board_outline2.41 (Q)
- net at R48.2: now also board_outline2.B1; no longer board_outline2.1 (GND)
- net at board_outline2.2 (I5): no longer R49.2
- net at board_outline2.4 (O5): no longer R51.2
- new net: R49.2, board_outline2.B3
- new net: R51.2, board_outline2.B4
Other:
- moved on the sheet: BAT1, D1, GPI1, ILI1, J14, R48, R49, R50, R51, R53, T108, T109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

Commit message: modularize
Parts:
- BAT1: footprint Connector_PinHeader_2.54mm:PinHeader_1x02_P2.54mm_Vertical -> project_fp:PinHeader_1x02_P2.54mm_Vertical_BAT
- J13, J16: LCSC (none) -> DNP; Package / Case (none) -> HEADER
- J15, J18, USB_DEVICE_1, USB_HOST_1, board_outline2: LCSC (none) -> DNP
Connections:
- net 3.3V: now also board_outline2.12 (3V), board_outline2.22 (3.3), board_outline2.30 (3V), board_outline2.40 (3V)
- net 5V: now also board_outline2.10 (5V), board_outline2.50 (5V)
- net ESP32_EN: now also board_outline2.56 (EN)
- net ESP32_IO0: now also board_outline2.60 (IOO)
- net ESP32_IO21_SDA: now also ESP_I1.1 (Pin_1), R20.2, R53.1; no longer R53.2, U2.33 (GPIO21)
- net ESP32_LED_OUT: now also board_outline2.44 (ESP)
- net GND: now also board_outline2.24 (G), board_outline2.32 (G), board_outline2.42 (GND), board_outline2.48 (G), board_outline2.58 (G), board_outline2.62 (BAT), board_outline2.8 (G)
- net GPIGPI1: now also board_outline2.20 (I1)
- net GPIO1: now also board_outline2.14 (IO1)
- net GPIO2: now also board_outline2.16 (IO2)
- net GPIO34: now also board_outline2.28 (34)
- net GPIO35: now also board_outline2.26 (35)
- net GPO1: now also board_outline2.18 (O1)
- net MIDI_IN_5: now also board_outline2.2 (I5)
- net MIDI_OUT_5: now also board_outline2.4 (O5)
- net MIDI_THRU_5: now also board_outline2.6 (T5)
- net OUTPUTA: now also board_outline2.34 (A36)
- net OUTPUTB: now also board_outline2.36 (B39)
- net SWITCH: now also board_outline2.38 (S27)
- net TEENSY_LED_OUT: now also board_outline2.46 (TSY)
- net T_BUTTON1: now also board_outline2.52 (?)
- net T_BUTTON2: now also board_outline2.54 (?)
- new net: R53.2, U2.33 (GPIO21)
Other:
- moved on the sheet: ESP_I1, H3, R20, R53
