File: t-dsp_desktop_pro.kicad_sch (KiCad schematic)
At the start: 194 parts, among them IC1 Logic Level Shifter - 74HCT2G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, J1 jumper, J10 JST-XH Connector, J11 JST-XH Connector, J12 RGB LED HEADEER, J13 Conn_01x02, J14 Conn_01x03, J15 Conn_01x01, J16 Conn_01x02, J17 Conn_02x04_Odd_Even, J18 Conn_02x02_Odd_Even, J19 Conn_01x01, J2 GROUND HEADER, J20 Conn_01x01, J21 jumper, J3 jumper, J4 jumper, J5 jumper, J6 jumper, J7 jumper, J8 PJRAS2X1S01X, J9 PJRAS2X1S01X, Q1 DMG2307L-7, Q2 DMG2307L-7, SW1 SW_SPST, SW2 TL1105WF160Q - 3.15mm actuator, SW3 SW_SPST, SW4 SW_SPST, SW5 RotaryEncoder_Switch_MP, SW6 TL1105WF160Q - 3.15mm actuator, SW7 TL1105WF160Q - 3.15mm actuator, SW8 TL1105WF160Q - 3.15mm actuator, T108 Tab, T109 Tab, T110 Tab, T111 Tab, U1 Teensy 4.1 - DEVKIT, U10 TPD4E02B04DQA, U2 ESP32-DevKitC - DEVKIT, U3 Power Mux & Protect - TPS2116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, U4 Optoisolators - H11L1SM - 6-S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, U5 Dual Buffer - SN74LVC2G125DCTR, U6 Dual Buffer - SN74LVC2G125DCTR, U7 Dual Buffer - SN74LVC2G125DCTR, U8 Dual Buffer - SN74LVC2G125DCTR, U9 Dual Buffer - 74HCT2G17GW,125

Commit message: v0.9-4layer: Add new components, 3D models, and board redesign for 4-layer stack
- Add footprints: 73725-0110BLF (RJ45), PRT-14417, SWITCHCRAFT_35RAPC4BV4, TPS22860DBVR
- Add 3D models: 35RAPC4BV4, 73725-0110BLF, 73725-11A0BLF, EC11E15204A3, PRT-14417, TPS22860DBVR, usb_A_vert
- Add schematic symbols: 35RAPC4BV4, 73725-0110BLF, 73725-11A0BLF, PRT-14417, TPS22860DBVR
- Update existing footprints: FCR6842032T, RJ45 Cetus, EC11E encoder, SK6812, expansion header, Teensy41, board outline, USB-A, ethernet header
- Major PCB layout update for 4-layer stackup
- Update schematic and project files

Co-Authored-By: Claude Sonnet 4.6 <noreply@anthropic.com>
Parts:
- added C36, C37: 0.1uF, project_fp:C_0805_2012Metric_Pad1.15x1.40mm_HandSolder, symbol TEENSY_4.0_ESP32_AUDIO-rescue:C_Small-Device
- added C38: 0.1uF, project_fp:C_0805_2012Metric_Pad1.15x1.40mm_HandSolder, symbol project_lib:CP1_Small-Device
- added C39: 30pF, project_fp:C_0805_2012Metric_Pad1.15x1.40mm_HandSolder, symbol TEENSY_4.0_ESP32_AUDIO-rescue:C_Small-Device
- added ETHERNET1: Ethernet Port - J1B1211CCD, project_fp:RJ45_Cetus_J1B1211CCD_Horizontal, symbol J1B1211CCD:J1B1211CCD
- added ETHERNET_J1: header, project_fp:ethernet_header, symbol ethernet_header:ethernet_header
- added G3: jumper, project_fp:SolderJumper-2_P1.3mm_Open_TrianglePad1.0x1.5mm, symbol Device:R
- added J22, J23: 35RAPC4BV4, project_fp:SWITCHCRAFT_35RAPC4BV4, symbol 35RAPC4BV4:35RAPC4BV4
- added J24: Conn_01x04, Connector_PinHeader_2.54mm:PinHeader_1x04_P2.54mm_Vertical, symbol Connector_Generic:Conn_01x04
- added J25: PRT-14417, project_fp:PRT-14417, symbol PRT-14417:PRT-14417
- added J26: 73725-0110BLF, project_fp:73725-0110BLF, symbol 73725-0110BLF:73725-0110BLF
- added SPDIF_IO2: header, project_fp:PinHeader_2x03_P2.54mm_Vertical, symbol Connector_Generic:Conn_02x03_Odd_Even
- added TR2: Optical Receiver - FCR6842032R, project_fp:FCR6842032T, symbol FCR6842032T(2):FCR6842032R
- added TT2: Optical Transmitter - FCR6842032T, project_fp:FCR6842032T, symbol FCR6842032T(2):FCR6842032T
- C7, C9, HPTRS1, HPTRS2, J18, J8, J9, J_PHONE1, MIDI_IN_1, USBA1, board_outline1: now left out of the parts list
- R25, R26: now not fitted; now left out of the parts list
- board_outline2: footprint project_fp:audio_project_board_outline_100x120 -> project_fp:audio_project_board_outline_100x100
Connections:
- net 14_SPDIF_OUT: now also J24.2 (Pin_2), SPDIF_IO2.3 (Pin_3), TT2.3 (VIN)
- net 15_SPDIF_IN: now also C39.1, J24.1 (Pin_1), SPDIF_IO2.1 (Pin_1), TR2.1 (VOUT)
- net 3.3V: now also C36.1, J24.3 (Pin_3), SPDIF_IO2.6 (Pin_6), TR2.3 (VCC)
- net 5V: now also C37.1, J24.4 (Pin_4), SPDIF_IO2.5 (Pin_5), TT2.2 (VCC)
- net GND: now also C36.2, C37.2, C38.2, C39.2, ETHERNET1.8 (GH_GND@1), ETHERNET1.9 (GRN-), ETHERNET_J1.2 (Pin_2), G3.2, SPDIF_IO2.2 (Pin_2), SPDIF_IO2.4 (Pin_4), TR2.2 (GND), TT2.1 (GND)
- net LED: now also ETHERNET1.10 (GRN+), ETHERNET_J1.3 (Pin_3)
- new net: J26.S1 (SHIELD), J26.S2 (SHIELD), J26.S3 (SHIELD), J26.S4 (SHIELD)
- new net: TR2.4 (NC), TR2.5 (NC)
- new net: C38.1, ETHERNET1.2 (TCT), ETHERNET1.5 (RCT)
- new net: TT2.4 (NC), TT2.5 (NC)
- new net: ETHERNET1.13 (CH_GND@2), ETHERNET1.14 (CH_GND@3), G3.1
- new net RX+: ETHERNET1.4 (RD+), ETHERNET_J1.1 (Pin_1)
- new net RX-: ETHERNET1.6 (RD-), ETHERNET_J1.4 (Pin_4)
- new net TX+: ETHERNET1.1 (TD+), ETHERNET_J1.6 (Pin_6)
- new net TX-: ETHERNET1.3 (TD-), ETHERNET_J1.5 (Pin_5)
- no-connect marks 18 -> 21
Other:
- note added: "ETHERNET"
