File: t-dsp_desktop_pro.kicad_sch (KiCad schematic)
At the start: 193 parts, among them IC1 Logic Level Shifter - 74HCT2G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, J1 jumper, J10 JST-XH Connector, J11 JST-XH Connector, J12 RGB LED HEADEER, J13 Conn_01x02, J14 Conn_01x03, J15 Conn_01x01, J16 Conn_01x02, J17 Conn_02x04_Odd_Even, J18 Conn_02x02_Odd_Even, J19 Conn_01x01, J2 GROUND HEADER, J20 Conn_01x01, J21 jumper, J3 jumper, J4 jumper, J5 jumper, J6 jumper, J7 jumper, J8 PJRAS2X1S01X, J9 PJRAS2X1S01X, Q1 DMG2307L-7, Q2 DMG2307L-7, SW1 SW_SPST, SW2 TL1105WF160Q - 3.15mm actuator, SW3 SW_SPST, SW4 SW_SPST, SW5 RotaryEncoder_Switch_MP, SW6 TL1105WF160Q - 3.15mm actuator, SW7 TL1105WF160Q - 3.15mm actuator, SW8 TL1105WF160Q - 3.15mm actuator, T108 Tab, T109 Tab, T110 Tab, T111 Tab, U1 Teensy 4.1 - DEVKIT, U10 TPD4E02B04DQA, U2 ESP32-DevKitC - DEVKIT, U3 Power Mux & Protect - TPS2116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, U4 Optoisolators - H11L1SM - 6-S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, U5 Dual Buffer - SN74LVC2G125DCTR, U6 Dual Buffer - SN74LVC2G125DCTR, U7 Dual Buffer - SN74LVC2G125DCTR, U8 Dual Buffer - SN74LVC2G125DCTR, U9 Dual Buffer - 74HCT2G17GW,125

Commit message: v0.8.4: Production release - final layout and schematic updates
Parts:
- added R54: 10k, project_fp:R_0805_2012Metric_Pad1.15x1.40mm_HandSolder, symbol Device:R
- R11: value 2.21k ohm -> 10k; LCSC C17520 -> C17414; LCSC_MPN 0805W8F2201T5E -> 0805W8F1002T5E
Connections:
- net 34_RX8_RESET2: now also R54.2
- net GND: now also R54.1
Other:
- moved on the sheet: J19, R11
Changed lines of the file:
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@@
 	)
 	(junction
-		(at 184.15 668.02)
+		(at 205.74 365.76)
 		(diameter 0)
 		(color 0 0 0 0)
 	)
 	(junction
-		(at 782.32 941.07)
+		(at 184.15 668.02)
 		(diameter 0)
 		(color 0 0 0 0)
 	)
 	(junction
-		(at 1045.21 372.11)
+		(at 782.32 941.07)
 		(diameter 0)
 		(color 0 0 0 0)
 	)
 	(junction
-		(at 195.58 363.22)
+		(at 1045.21 372.11)
 		(diameter 0)
 		(color 0 0 0 0)
@@
 	)
 	(junction
+		(at 204.47 363.22)
+		(diameter 0)
+		(color 0 0 0 0)
+	)
+	(junction
 		(at 1056.64 412.75)
 		(diameter 0)
@@
 	(wire
 		(pts
+			(xy 204.47 363.22) (xy 207.01 363.22)
+		)
+		(stroke
+			(width 0)
+			(type default)
+		)
+	)
+	(wire
+		(pts
 			(xy 99.06 368.3) (xy 105.41 368.3)
 		)
@@
 	(wire
 		(pts
-			(xy 195.58 363.22) (xy 207.01 363.22)
-		)
-		(stroke
-			(width 0)
-			(type default)
-		)
-	)
-	(wire
-		(pts
 			(xy 335.28 306.07) (xy 339.09 306.07)
 		)
@@
 	(wire
 		(pts
-			(xy 187.96 370.84) (xy 187.96 368.3)
+			(xy 187.96 382.27) (xy 187.96 368.3)
 		)
 		(stroke
@@
 	(wire
 		(pts
-			(xy 207.01 365.76) (xy 161.29 365.76)
+			(xy 207.01 365.76) (xy 205.74 365.76)
 		)
 		(stroke
@@
 	(wire
 		(pts
+			(xy 205.74 365.76) (xy 161.29 365.76)
+		)
+		(stroke
+			(width 0)
+			(type default)
+		)
+	)
+	(wire
+		(pts
 			(xy 494.03 899.16) (xy 501.65 899.16)
 		)
@@
 	(wire
 		(pts
-			(xy 189.23 370.84) (xy 187.96 370.84)
+			(xy 189.23 382.27) (xy 187.96 382.27)
 		)
 		(stroke
@@
 	(wire
 		(pts
+			(xy 205.74 365.76) (xy 205.74 368.3)
+		)
+		(stroke
+			(width 0)
+			(type default)
+		)
+	)
+	(wire
+		(pts
 			(xy 1163.32 862.33) (xy 1163.32 864.87)
 		)
@@
 	(wire
 		(pts
+			(xy 204.47 360.68) (xy 204.47 363.22)
+		)
+		(stroke
+			(width 0)
+			(type default)
+		)
+	)
+	(wire
+		(pts
 			(xy 228.6 596.9) (xy 252.73 596.9)
 		)
@@
 	(wire
 		(pts
-			(xy 195.58 363.22) (xy 161.29 363.22)
+			(xy 161.29 363.22) (xy 204.47 363.22)
 		)
 		(stroke
@@
 	(global_label "GND"
 		(shape input)
-		(at 185.42 374.65 180)
+		(at 198.12 368.3 180)
 		(fields_autoplaced yes)
 		(effects
@@
 		)
 		(property "Intersheetrefs" "${INTERSHEET_REFS}"
-			(at 270.51 454.66 0)
+			(at 283.21 448.31 0)
 			(effects
 				(font
@@
 	(global_label "3.3V"
 		(shape input)
-		(at 195.58 355.6 180)
+		(at 196.85 360.68 180)
 		(fields_autoplaced yes)
 		(effects
@@
 		)
 		(property "Intersheetrefs" "${INTERSHEET_REFS}"
-			(at 189.1434 355.6794 0)
+			(at 189.7524 360.68 0)
 			(effects
 				(font
@@
 	)
 	(symbol
+		(lib_id "Device:R")
+		(at 201.93 368.3 90)
+		(unit 1)
+		(exclude_from_sim no)
+		(in_bom yes)
+		(on_board yes)
+		(dnp no)
+		(property "Reference" "R54"
+			(at 201.93 368.3 90)
+			(effects
+				(font
+					(size 0.9906 0.9906)
+				)
+			)
+		)
+		(property "Value" "10k"
+			(at 202.438 371.094 90)
+			(effects
+				(font
+					(size 1.27 1.27)
+				)
+			)
+		)
+		(property "Footprint" "project_fp:R_0805_2012Metric_Pad1.15x1.40mm_HandSolder"
+			(at 201.93 370.078 90)
+			(effects
+				(font
+					(size 1.27 1.27)
+				)
+				(hide yes)
+			)
+		)
+		(property "Datasheet" ""
+			(at 201.93 368.3 0)
+			(effects
+				(font
+					(size 1.27 1.27)
+				)
+				(hide yes)
+			)
+		)
+		(property "Description" "10kΩ ±1% 125mW 0805 Thick Film Resistor"
+			(at 201.93 368.3 0)
+			(effects
+				(font
+					(size 1.27 1.27)
+				)
+				(hide yes)
+			)
+		)
+		(property "Package / Case" "R0805"
+			(at 201.93 368.3 0)
+			(effects
+				(font
+					(size 1.27 1.27)
+				)
+				(hide yes)
+			)
+		)
+		(property "LCSC" "C17414"
+			(at 201.93 368.3 0)
+			(effects
+				(font
+					(size 1.27 1.27)
+				)
+				(hide yes)
+			)
+		)
+		(property "LCSC TYPE" "SMD"
+			(at 201.93 368.3 0)
+			(effects
+				(font
+					(size 1.27 1.27)
+				)
+				(hide yes)
+			)
+		)
+		(property "LCSC_MPN" "0805W8F1002T5E"
+			(at 201.93 368.3 0)
+			(effects
+				(font
+					(size 1.27 1.27)
+				)
+				(hide yes)
+			)
+		)
+		(property "LCSC_Manufacturer" "UNI-ROYAL"
+			(at 201.93 368.3 0)
+			(effects
+				(font
+					(size 1.27 1.27)
+				)
+				(hide yes)
+			)
+		)
+		(pin "1"
+		)
+		(pin "2"
+		)
+		(instances
+			(project "t-dsp_desktop_pro"
+				(path "/6a0ff39d-771d-410f-9e7c-006586d81d16"
+					(reference "R54")
+					(unit 1)
+				)
+			)
+		)
+	)
+	(symbol
 		(lib_id "proejct_lib:R_Small")
 		(at 215.9 321.31 270)
@@
 	(symbol
 		(lib_id "Device:R")
-		(at 195.58 359.41 0)
+		(at 200.66 360.68 90)
 		(unit 1)
 		(exclude_from_sim no)
@@
 		(dnp no)
 		(property "Reference" "R11"
-			(at 200.025 357.505 0)
+			(at 200.914 360.68 90)
 			(effects
 				(font
@@
 			)
 		)
-		(property "Value" "2.21k ohm"
-			(at 209.55 359.41 0)
+		(property "Value" "10k"
+			(at 200.406 358.394 90)
 			(effects
 				(font
@@
 		)
 		(property "Footprint" "project_fp:R_0805_2012Metric_Pad1.15x1.40mm_HandSolder"
-			(at 193.802 359.41 90)
+			(at 200.66 362.458 90)
 			(effects
 				(font
@@
 		)
 		(property "Datasheet" ""
-			(at 195.58 359.41 0)
+			(at 200.66 360.68 0)
 			(effects
 				(font
@@
 			)
 		)
-		(property "Description" "2.2kΩ ±1% 125mW 0805 Thick Film Resistor"
-			(at 195.58 359.41 0)
+		(property "Description" "10kΩ ±1% 125mW 0805 Thick Film Resistor"
+			(at 200.66 360.68 0)
 			(effects
 				(font
@@
 		)
 		(property "Package / Case" "R0805"
-			(at 195.58 359.41 0)
+			(at 200.66 360.68 0)
 			(effects
 				(font
@@
 			)
 		)
-		(property "LCSC" "C17520"
-			(at 195.58 359.41 0)
+		(property "LCSC" "C17414"
+			(at 200.66 360.68 0)
 			(effects
 				(font
@@
 		)
 		(property "LCSC TYPE" "SMD"
-			(at 195.58 359.41 0)
+			(at 200.66 360.68 0)
 			(effects
 				(font
@@
 			)
 		)
-		(property "LCSC_MPN" "0805W8F2201T5E"
-			(at 195.58 359.41 0)
+		(property "LCSC_MPN" "0805W8F1002T5E"
+			(at 200.66 360.68 0)
 			(effects
 				(font
@@
 		)
 		(property "LCSC_Manufacturer" "UNI-ROYAL"
-			(at 195.58 359.41 0)
+			(at 200.66 360.68 0)
 			(effects
 				(font
@@
 	(symbol
 		(lib_id "Connector_Generic:Conn_01x01")
-		(at 194.31 370.84 0)
+		(at 194.31 382.27 0)
 		(unit 1)
 		(exclude_from_sim no)
@@
 		(fields_autoplaced yes)
 		(property "Reference" "J19"
-			(at 196.85 369.5699 0)
+			(at 196.85 380.9999 0)
 			(effects
 				(font
@@
 		)
 		(property "Value" "Conn_01x01"
-			(at 196.85 372.1099 0)
+			(at 196.85 383.5399 0)
 			(effects
 				(font
@@
 		)
 		(property "Footprint" "project_fp:OUT1B_PinHeader_1x01_P2.54mm_Vertical"
-			(at 194.31 370.84 0)
+			(at 194.31 382.27 0)
 			(effects
 				(font
@@
 		)
 		(property "Datasheet" "~"
-			(at 194.31 370.84 0)
+			(at 194.31 382.27 0)
 			(effects
 				(font
@@
 		)
 		(property "Description" "Generic connector, single row, 01x01, script generated (kicad-library-utils/schlib/autogen/connector/)"
-			(at 194.31 370.84 0)
+			(at 194.31 382.27 0)
 			(effects
 				(font
@@
 		)
 		(property "Package / Case" "HEADER"
-			(at 194.31 370.84 0)
+			(at 194.31 382.27 0)
 			(effects
 				(font
@@
 		)
 		(property "LCSC" "DNP"
-			(at 194.31 370.84 0)
+			(at 194.31 382.27 0)
 			(effects
 				(font
@@
 		)
 		(property "LCSC_MPN" ""
-			(at 194.31 370.84 0)
+			(at 194.31 382.27 0)
 			(effects
 				(font
@@
 		)
 		(property "LCSC_Manufacturer" ""
-			(at 194.31 370.84 0)
+			(at 194.31 382.27 0)
 			(effects
 				(font

Commit message: update
Parts:
- removed C11: 0.1uF, project_fp:C_0805_2012Metric_Pad1.15x1.40mm_HandSolder, symbol TEENSY_4.0_ESP32_AUDIO-rescue:C_Small-Device
- added C36, C37, C40: 0.1uF, project_fp:C_0805_2012Metric_Pad1.15x1.40mm_HandSolder, symbol TEENSY_4.0_ESP32_AUDIO-rescue:C_Small-Device
- added C38: 0.1uF, project_fp:C_0805_2012Metric_Pad1.15x1.40mm_HandSolder, symbol project_lib:CP1_Small-Device
- added C39: 30pF, project_fp:C_0805_2012Metric_Pad1.15x1.40mm_HandSolder, symbol TEENSY_4.0_ESP32_AUDIO-rescue:C_Small-Device
- added ETHERNET1: Ethernet Port - J1B1211CCD, project_fp:RJ45_Cetus_J1B1211CCD_Horizontal, symbol J1B1211CCD:J1B1211CCD
- added ETHERNET_J1: header, project_fp:ethernet_header, symbol ethernet_header:ethernet_header
- added G3: jumper, project_fp:SolderJumper-2_P1.3mm_Open_TrianglePad1.0x1.5mm, symbol Device:R
- added J22, J23: 35RAPC4BV4, project_fp:SWITCHCRAFT_35RAPC4BV4, symbol 35RAPC4BV4:35RAPC4BV4
- added J24: Conn_01x04, Connector_PinHeader_2.54mm:PinHeader_1x04_P2.54mm_Vertical, symbol Connector_Generic:Conn_01x04
- added J25: PRT-14417, project_fp:PRT-14417, symbol PRT-14417:PRT-14417
- added J26: 73725-0110BLF, project_fp:73725-0110BLF, symbol 73725-0110BLF:73725-0110BLF
- added J27: Conn_01x04, project_fp:Teensy41_board_outline, symbol Connector_Generic:Conn_01x04
- added MK1, MK2: SPK0641HT4H-1, project_fp:SPK0641HT4H-1, symbol SPK0641HT4H-1:SPK0641HT4H-1
- added SPDIF_IO2: header, project_fp:PinHeader_2x03_P2.54mm_Vertical, symbol Connector_Generic:Conn_02x03_Odd_Even
- added TR2: Optical Receiver - FCR6842032R, project_fp:FCR6842032T, symbol FCR6842032T(2):FCR6842032R
- added TT2: Optical Transmitter - FCR6842032T, project_fp:FCR6842032T, symbol FCR6842032T(2):FCR6842032T
- C7, C9: footprint project_fp:CP_Radial_D10.0mm_P5.00mm_AND_D8.0mm_P3.5mm -> Capacitor_THT:CP_Radial_D6.3mm_P2.50mm; now left out of the parts list
- HPTRS1, HPTRS2, J18, J8, J9, J_PHONE1, MIDI_IN_1: now left out of the parts list
- R12: footprint project_fp:R_0805_2012Metric_Pad1.15x1.40mm_HandSolder -> project_fp:jumper_slice
- R25, R26: now not fitted; now left out of the parts list
- U1: footprint project_fp:Teensy41_mod3 -> project_fp:Teensy41_simple
- USBA1: footprint project_fp:TE_292303-5_USB_A -> project_fp:TE_292303-5_USB_A_tight_fit; now left out of the parts list
- board_outline1: footprint project_fp:audio_module_board_outline_50x34.5_d1 -> project_fp:audio_module_board_outline_50x34.5_d1_ADAPTOR; now left out of the parts list
- board_outline2: footprint project_fp:audio_project_board_outline_100x120 -> project_fp:audio_project_board_outline_100x100
Connections:
- net 14_SPDIF_OUT: now also J24.2 (Pin_2), SPDIF_IO2.3 (Pin_3), TT2.3 (VIN)
- net 15_SPDIF_IN: now also C39.1, J24.1 (Pin_1), SPDIF_IO2.1 (Pin_1), TR2.1 (VOUT)
- net 3.3V: now also C36.1, C40.1, J24.3 (Pin_3), MK1.3 (SELECT), MK1.4 (VDD), MK2.4 (VDD), SPDIF_IO2.6 (Pin_6), TR2.3 (VCC); no longer MIC1.5 (VDD), MIC2.5 (VDD)
- net 35_TX8_RESET: now also U1.14 (12_MISO_MQSL); no longer U1.27 (35_TX8)
- net 5V: now also C37.1, J24.4 (Pin_4), SPDIF_IO2.5 (Pin_5), TT2.2 (VCC)
- net 7_OUT1A: now also board_outline1.7 (DSP_DOUT)
- net 7_OUT1A+: no longer board_outline1.7 (DSP_DOUT)
- net 9_OUT1C_INPUT: no longer U1.11 (9_OUT1C)
- net BCLK1: now also board_outline1.11 (BCLK)
- net BCLK1+TDM1: no longer board_outline1.11 (BCLK)
- net GND: now also C36.2, C37.2, C38.2, C39.2, C40.2, ETHERNET1.8 (GH_GND@1), ETHERNET1.9 (GRN-), ETHERNET_J1.2 (Pin_2), G3.2, MK1.5 (GND), MK1.6 (GND), MK1.7 (GND), MK1.8 (GND), MK2.3 (SELECT), MK2.5 (GND), MK2.6 (GND), MK2.7 (GND), MK2.8 (GND), SPDIF_IO2.2 (Pin_2), SPDIF_IO2.4 (Pin_4), TR2.2 (GND), TT2.1 (GND)
- net GPIGPI1: now also MK1.1 (DATA), MK2.1 (DATA); no longer MIC1.1 (DATA), MIC2.1 (DATA)
- net GPIO1: now also MK1.2 (CLOCK), MK2.2 (CLOCK); no longer MIC1.4 (LRCLK-WS-FS), MIC2.4 (LRCLK-WS-FS)
- net LED: now also ETHERNET1.10 (GRN+), ETHERNET_J1.3 (Pin_3)
- net LRCK1: now also board_outline1.13 (LRCK)
- net LRCK1+TDM1: no longer board_outline1.13 (LRCK)
- net at MIC2.4 (LRCLK-WS-FS): now also MIC1.4 (LRCLK-WS-FS)
- net ESP32_IO12_SPI_MISO renamed ESP32_IO12_VSPI_MISO
- net ESP32_IO12_VSPI_MISO: no longer U1.14 (12_MISO_MQSL)
- net ESP32_IO13_SPI_MOSI renamed ESP32_IO13_VSPI_MOSI
- net ESP32_IO13_VSPI_MOSI: no longer U1.13 (11_MOSI_CTX1)
- net ESP32_IO33_SPI_CS renamed ESP32_IO17_VSPI_CS
- net ESP32_IO17_VSPI_CS: no longer U1.12 (10_CS_MQSR)
- new net: J26.S1 (SHIELD), J26.S2 (SHIELD), J26.S3 (SHIELD), J26.S4 (SHIELD)
- new net: TR2.4 (NC), TR2.5 (NC)
- new net: C38.1, ETHERNET1.2 (TCT), ETHERNET1.5 (RCT)
- new net: TT2.4 (NC), TT2.5 (NC)
- new net: ETHERNET1.13 (CH_GND@2), ETHERNET1.14 (CH_GND@3), G3.1
- new net RX+: ETHERNET1.4 (RD+), ETHERNET_J1.1 (Pin_1)
- new net RX-: ETHERNET1.6 (RD-), ETHERNET_J1.4 (Pin_4)
- new net TX+: ETHERNET1.1 (TD+), ETHERNET_J1.6 (Pin_6)
- new net TX-: ETHERNET1.3 (TD-), ETHERNET_J1.5 (Pin_5)
- no-connect marks 18 -> 21
Other:
- note added: "ETHERNET"
- moved on the sheet: BAT1, BAT2, C10, C2, C3, C6, C7, C8, C9, D1, HPTRS1, HPTRS2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
