File: t-dsp_desktop_pro.kicad_pcb (KiCad board)
At the start: 8 copper layers, 120 x 100 mm, 154 parts, among them IC1 Logic Level Shifter - 74HCT2G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, J1 jumper, J10 JST-XH Connector -, J11 JST-XH Connector -, J12 RGB LED HEADEER, J13 Conn_01x02, J15 Conn_01x01, J16 Conn_01x02, J17 Conn_02x04_Odd_Even, J18 Conn_02x02_Odd_Even, J19 Conn_01x01, J2 GROUND HEADER, J20 Conn_01x01, J3 jumper, J4 jumper, J5 jumper, J6 jumper, J7 jumper, J8 PJRAS2X1S01X, J9 PJRAS2X1S01X, Q1 DMG2307L-7, Q2 DMG2307L-7, T108 Tab, T109 Tab, T110 Tab, T111 Tab, U1 Teensy 4.1 - DEVKIT, U10 TPD4E02B04DQA, U2 ESP32-DevKitC - DEVKIT, U3 Power Mux & Protect - TPS2116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, U4 Optoisolators - H11L1SM - 6-S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, U5 Dual Buffer - SN74LVC2G125DCTR, U6 Dual Buffer - SN74LVC2G125DCTR, U7 Dual Buffer - SN74LVC2G125DCTR, U8 Dual Buffer - SN74LVC2G125DCTR, U9 Dual Buffer - 74HCT2G17GW,125

Commit message: v0.81: Fix CI release, localize 3D models, update README with render gallery
- Fix workflow: add gh release create before upload (tag != release)
- Fix ZIP filename: remove empty %r board revision from output name
- Localize 3D model paths for U10, C15, JST connectors to ${KIPRJMOD}
- Add project-local footprints for C_1206 and JST_XH_S2B-XH-A
- Trim SMD 3D renders from 8 to 4 views (top, bottom, top_iso, bottom_iso)
- Update gallery.html to handle different view counts per set
- Update README: Blender render thumbnails linking to gallery, fix IC table,
  add new components (U10, IC1, D5, Q1/Q2), update project files table
Parts:
- C15: footprint Capacitor_SMD:C_1206_3216Metric_Pad1.33x1.80mm_HandSolder -> project_fp:C_1206_3216Metric_Pad1.33x1.80mm_HandSolder
- J10, J11: value JST-XH Connector - -> JST-XH Connector; footprint Connector_JST:JST_XH_S2B-XH-A_1x02_P2.50mm_Horizontal -> project_fp:JST_XH_S2B-XH-A_1x02_P2.50mm_Horizontal
- U10: footprint Package_SON:USON-10_2.5x1.0mm_P0.5mm -> project_fp:TPD4E02B04DQA
