File: panel/jlcpcb_1x1/jlcpcb_1x1.kicad_pcb (KiCad board)
At the start: 8 copper layers, 134 x 114 mm, 144 parts, among them IC1 74HCT2G125DC,125, J1 jumper, J10 JST-XH Connector, J11 JST-XH Connector, J2 Conn_01x01_Pin, J3 jumper, J4 jumper, J5 jumper, J6 jumper, J7 jumper, J8 PJRAS2X1S01X, J9 PJRAS2X1S01X, U1 Teensy 4.1 - DEVKIT, U2 ESP32-DevKitC - DEVKIT, U3 TPS2116DRL, U4 Optoisolators - H11L1SM - 6-S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, U5 SN74LVC2G125DCTR, U6 SN74LVC2G125DCTR, U7 SN74LVC2G125DCTR, U8 SN74LVC2G125DCTR, U9 Dual Buffer - 74HCT2G17GW,125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

Commit message: update
Parts:
- removed D5: HEADER, project_fp:LED_GPIO_PinHeader_1x04_P2.54mm_Vertical
- added J12: RGB LED HEADEER, project_fp:LED_GPIO_PinHeader_1x04_P2.54mm_Vertical, F.Cu at (271.4, 95.3)
- added R40: 49.9 ohm, project_fp:R_0805_2012Metric_Pad1.15x1.40mm_HandSolder, F.Cu at (204.4, 74.0)
- added R41: 49.9 ohm, project_fp:R_0805_2012Metric_Pad1.15x1.40mm_HandSolder, F.Cu at (212.9, 73.5)
- added R42: 49.9 ohm, project_fp:R_0805_2012Metric_Pad1.15x1.40mm_HandSolder, F.Cu at (212.9, 86.0)
- added R43: 49.9 ohm, project_fp:R_0805_2012Metric_Pad1.15x1.40mm_HandSolder, F.Cu at (203.9, 86.0)
- added R44: 49.9 ohm, project_fp:R_0805_2012Metric_Pad1.15x1.40mm_HandSolder, F.Cu at (212.9, 80.0)
- added R45: 49.9 ohm, project_fp:R_0805_2012Metric_Pad1.15x1.40mm_HandSolder, F.Cu at (203.9, 80.0)
- added R46: 49.9 ohm, project_fp:R_0805_2012Metric_Pad1.15x1.40mm_HandSolder, F.Cu at (212.9, 92.0)
- added R47: 49.9 ohm, project_fp:R_0805_2012Metric_Pad1.15x1.40mm_HandSolder, F.Cu at (203.9, 92.0)
- added R48: 0 ohm, project_fp:R_0805_2012Metric_Pad1.15x1.40mm_HandSolder, F.Cu at (160.9, 39.0)
- added R49: 0 ohm, project_fp:R_0805_2012Metric_Pad1.15x1.40mm_HandSolder, F.Cu at (164.9, 121.0)
- added R50: 0 ohm, project_fp:R_0805_2012Metric_Pad1.15x1.40mm_HandSolder, F.Cu at (267.4, 33.5)
- added R51: 0 ohm, project_fp:R_0805_2012Metric_Pad1.15x1.40mm_HandSolder, F.Cu at (271.4, 116.5)
- BAT1: value BAT -> BAT HEADER
- C1: value 1uF -> 1 uF
- C12, C13, C23: value 10uF -> 10 uF
- C14, C16, C17, C18, C19, C2, C20, C21, C22, C3, C4, C5: value 0.1uF -> 0.1 uF
- C15: value 100uF -> 100 uF
- C7, C9: value 470uF Electrolytic -> 470 uF Electrolytic Audio-Grade
- CC1, CC2, R30: value 5.1k -> 5.1k ohm; footprint project_fp:R_0805_2012Metric_Pad1.20x1.40mm_HandSolder -> project_fp:R_0805_2012Metric_Pad1.15x1.40mm_HandSolder
- D3, D4: value SK6812 -> Side Light LED - SK6812
- ESP_I1: value header -> ESP32 I2C HEADER
- GPI1: value header -> ESP32 GPI HEADER
- HPTRS1, HPTRS2: value 3.5MM JACK -> 3.5mm TRS - 35RAPC3BH3
- IC1: value 74HCT2G125DC,125 -> Logic Level Shifter - 74HCT2G125DC,125
- J10, J11: value JST-XH Connector -> JST-EH Connector - S02B-PASK-2; footprint Connector_JST:JST_EH_S2B-EH_1x02_P2.50mm_Horizontal -> project_fp:JST_EH_S2B-EH_1x02_P2.50mm_Horizontal
- J2: value Conn_01x01_Pin -> GROUND HEADER
- PWR1, PWR2: value LED_1206 -> LED Power Indicator - 1206 5v 2.0 V Forward
- R1, R2, R5, R6, R7, R9: value 100 ohm -> 49.9 ohm; footprint project_fp:R_0805_2012Metric_Pad1.20x1.40mm_HandSolder -> project_fp:R_0805_2012Metric_Pad1.15x1.40mm_HandSolder
- R10: value 100 ohm -> 49.9 ohm
- R11, R19, R20, R21, R22, R23: value 2.2k ohm - 2200 ohm -> 2.21k ohm; footprint project_fp:R_0805_2012Metric_Pad1.20x1.40mm_HandSolder -> project_fp:R_0805_2012Metric_Pad1.15x1.40mm_HandSolder
- R13, R14, R16, R17: footprint Resistor_SMD:R_0402_1005Metric_Pad0.72x0.64mm_HandSolder -> project_fp:R_0805_2012Metric_Pad1.15x1.40mm_HandSolder
- R18, R8: value 470 ohm -> 220 ohm
- R25, R26: value 22 ohm -> 49.9 ohm; footprint project_fp:R_0805_2012Metric_Pad1.20x1.40mm_HandSolder -> project_fp:R_0805_2012Metric_Pad1.15x1.40mm_HandSolder
- R28: value 16.9k -> 16.9k ohm; footprint project_fp:R_0805_2012Metric_Pad1.20x1.40mm_HandSolder -> project_fp:R_0805_2012Metric_Pad1.15x1.40mm_HandSolder
- R29: value 5.00k -> 5.1k ohm; footprint project_fp:R_0805_2012Metric_Pad1.20x1.40mm_HandSolder -> project_fp:R_0805_2012Metric_Pad1.15x1.40mm_HandSolder
- R3, R4: footprint project_fp:R_0805_2012Metric_Pad1.20x1.40mm_HandSolder -> project_fp:R_0805_2012Metric_Pad1.15x1.40mm_HandSolder
- R31, R35: value 0ohm -> 0 ohm; footprint project_fp:R_0805_2012Metric_Pad1.20x1.40mm_HandSolder -> project_fp:R_0805_2012Metric_Pad1.15x1.40mm_HandSolder
- R33: value 1.5k -> 1.5k ohm; footprint project_fp:R_0805_2012Metric_Pad1.20x1.40mm_HandSolder -> project_fp:R_0805_2012Metric_Pad1.15x1.40mm_HandSolder
- R36, R39: value 47 ohm -> 220 ohm
- RLED1, RLED2: value led -> 2.21k ohm; footprint project_fp:R_0805_2012Metric_Pad1.20x1.40mm_HandSolder -> project_fp:R_0805_2012Metric_Pad1.15x1.40mm_HandSolder
- TDM1, TDM2: value header -> I2S /I2C EXPANSION HEADER
- T_PROG1: value header -> TEENSY SWITCH HEADER
- U3: value TPS2116DRL -> Power Mux & Protect - TPS2116DRL
- U5, U6, U7, U8: value SN74LVC2G125DCTR -> Dual Buffer - SN74LVC2G125DCTR
- U9: value Dual Buffer - 74HCT2G17GW,125 - SOT-363_SC-70-6 -> Dual Buffer - 74HCT2G17GW,125
- USBC1: value USB C Device - USB4085-GF-A -> USB C Port - Through Hole USB4085-GF-A
- moved PWR2 2.50 mm to (199.9, 47.5)
- moved RLED2 2.50 mm to (199.9, 51.5), turned to 180 degrees
- moved R15 1.24 mm to (226.4, 89.0)
- moved R17 0.71 mm to (226.4, 94.0)
- moved R16 0.50 mm to (226.4, 91.5)
- moved R12 0.07 mm to (217.4, 59.4)
Connections:
- R12 pad 2: Board_0-IOVDD -> Board_0-3.3V
- U5 pad 3: Board_0-LRCK1+TDM2 -> Board_0-Net-(U5-2Y)
- U5 pad 6: Board_0-LRCK1+TDM1 -> Board_0-Net-(U5-1Y)
- U6 pad 3: Board_0-MCLK1+TDM2 -> Board_0-Net-(U6-2Y)
- U6 pad 6: Board_0-MCLK1+TDM1 -> Board_0-Net-(U6-1Y)
- U7 pad 3: Board_0-BCLK1+TDM2 -> Board_0-Net-(U7-2Y)
- U7 pad 4: Board_0-unconnected-(U7-GND-Pad4) -> Board_0-GND
- U7 pad 6: Board_0-BCLK1+TDM1 -> Board_0-Net-(U7-1Y)
- U8 pad 3: Board_0-6_OUT1D+ -> Board_0-Net-(U8-2Y)
- U8 pad 4: Board_0-unconnected-(U8-GND-Pad4) -> Board_0-GND
- U8 pad 6: Board_0-7_OUT1A+ -> Board_0-Net-(U8-1Y)
- board_outline2 pad 1: Board_0-unconnected-(board_outline2-GND-Pad1) -> Board_0-Net-(R48-Pad2)
- board_outline2 pad 2: Board_0-unconnected-(board_outline2-GND-Pad2) -> Board_0-Net-(R49-Pad2)
- board_outline2 pad 3: Board_0-unconnected-(board_outline2-GND-Pad3) -> Board_0-Net-(R50-Pad2)
- board_outline2 pad 4: Board_0-unconnected-(board_outline2-GND-Pad4) -> Board_0-Net-(R51-Pad2)
Routing:
- net Board_0-GND: track 116.0 -> 441.4 mm, vias 191 -> 227
- net Board_0-Net-(HPTRS2-Pad4): track 93.7 -> 147.4 mm, vias 0 -> 1
- net Board_0-Net-(HPTRS2-Pad3): track 115.0 -> 166.9 mm, vias 0 -> 1
- net Board_0-Net-(HPTRS1-Pad4): track 148.8 -> 118.9 mm, vias 1 -> 2
- net Board_0-/AUDIO_OUT2P: track 35.2 -> 53.4 mm, vias 0 -> 1
- net Board_0-3.3V: track 331.2 -> 348.0 mm, vias 13 -> 14
- net Board_0-/AUDIO_OUTP: track 38.4 -> 54.4 mm, vias 0 -> 1
- net Board_0-/AUDIO_IN2P: track 50.0 -> 61.8 mm, vias 0 -> 1
- net Board_0-Net-(HPTRS1-Pad3): track 94.9 -> 104.9 mm, vias 1 -> 2
- net Board_0-Net-(1/4-PHONE1-PadT): track 39.8 -> 47.2 mm, vias 0 -> 1
- net Board_0-Net-(1/4-PHONE1-PadR): track 26.1 -> 33.2 mm, vias 0 -> 1
- net Board_0-Net-(R49-Pad2): track 0.00 -> 6.60 mm
- net Board_0-Net-(R48-Pad2): track 0.00 -> 6.57 mm
- net Board_0-SDA0: track 116.8 -> 123.1 mm
- net Board_0-6_OUT1D+: track 51.2 -> 45.1 mm
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