File: panel/jlcpcb_1x1/jlcpcb_1x1.kicad_pcb (KiCad board)
At the start: 8 copper layers, 134 x 114 mm, 156 parts, among them IC1 Logic Level Shifter - 74HCT2G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, J1 jumper, J10 JST-EH Connector - S02B-PASK-2, J11 JST-EH Connector - S02B-PASK-2, J12 RGB LED HEADEER, J2 GROUND HEADER, J3 jumper, J4 jumper, J5 jumper, J6 jumper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

Commit message: update
Parts:
- removed KiKit_MB_1_6, KiKit_MB_1_7, KiKit_MB_2_6, KiKit_MB_2_7, KiKit_MB_3_6, KiKit_MB_3_7, KiKit_MB_4_6, KiKit_MB_4_7: NPTH, NPTH
- added KiKit_MB_5_2: NPTH, NPTH, F.Cu at (149.3, 27.0)
- added KiKit_MB_5_3: NPTH, NPTH, F.Cu at (150.1, 27.0)
- added KiKit_MB_5_4: NPTH, NPTH, F.Cu at (151.0, 27.0)
- added KiKit_MB_5_5: NPTH, NPTH, F.Cu at (151.8, 27.0)
- added KiKit_MB_5_6: NPTH, NPTH, F.Cu at (152.7, 27.0)
- added KiKit_MB_5_7: NPTH, NPTH, F.Cu at (153.5, 27.0)
- added KiKit_MB_6_2: NPTH, NPTH, F.Cu at (149.3, 127.0)
- added KiKit_MB_6_3: NPTH, NPTH, F.Cu at (150.1, 127.0)
- added KiKit_MB_6_4: NPTH, NPTH, F.Cu at (151.0, 127.0)
- added KiKit_MB_6_5: NPTH, NPTH, F.Cu at (151.8, 127.0)
- added KiKit_MB_6_6: NPTH, NPTH, F.Cu at (152.7, 127.0)
- added KiKit_MB_6_7: NPTH, NPTH, F.Cu at (153.5, 127.0)
- added KiKit_MB_7_2: NPTH, NPTH, F.Cu at (278.3, 27.0)
- added KiKit_MB_7_3: NPTH, NPTH, F.Cu at (279.1, 27.0)
- added KiKit_MB_7_4: NPTH, NPTH, F.Cu at (280.0, 27.0)
- added KiKit_MB_7_5: NPTH, NPTH, F.Cu at (280.8, 27.0)
- added KiKit_MB_7_6: NPTH, NPTH, F.Cu at (281.7, 27.0)
- added KiKit_MB_7_7: NPTH, NPTH, F.Cu at (282.5, 27.0)
- added KiKit_MB_8_2: NPTH, NPTH, F.Cu at (278.3, 127.0)
- added KiKit_MB_8_3: NPTH, NPTH, F.Cu at (279.1, 127.0)
- added KiKit_MB_8_4: NPTH, NPTH, F.Cu at (280.0, 127.0)
- added KiKit_MB_8_5: NPTH, NPTH, F.Cu at (280.8, 127.0)
- added KiKit_MB_8_6: NPTH, NPTH, F.Cu at (281.7, 127.0)
- added KiKit_MB_8_7: NPTH, NPTH, F.Cu at (282.5, 127.0)
- moved KiKit_MB_2_2 150.6 mm to (276.1, 45.8)
- moved KiKit_MB_2_3 149.5 mm to (276.1, 46.6)
- moved KiKit_MB_2_4 148.3 mm to (276.1, 47.4)
- moved KiKit_MB_2_5 147.2 mm to (276.1, 48.2)
- moved KiKit_MB_4_5 127.0 mm to (155.7, 105.8)
- moved KiKit_MB_4_4 126.0 mm to (155.7, 106.6)
- moved KiKit_MB_4_3 125.0 mm to (155.7, 107.4)
- moved KiKit_MB_4_2 124.0 mm to (155.7, 108.2)
- moved KiKit_MB_3_5 81.3 mm to (276.1, 108.2)
- moved KiKit_MB_3_4 80.5 mm to (276.1, 107.4)
- moved KiKit_MB_3_3 79.7 mm to (276.1, 106.6)
- moved KiKit_MB_3_2 78.8 mm to (276.1, 105.8)
- moved KiKit_MB_1_2 22.1 mm to (155.7, 48.2)
- moved KiKit_MB_1_3 21.1 mm to (155.7, 47.4)
- moved KiKit_MB_1_4 20.2 mm to (155.7, 46.6)
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Other:
- outline, holes or cut-outs redrawn
