File: panel/jlcpcb_1x1/jlcpcb_1x1.kicad_pcb (KiCad board)
At the start: 8 copper layers, 134 x 114 mm, 172 parts, among them IC1 Logic Level Shifter - 74HCT2G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, J1 jumper, J10 JST-EH Connector - S02B-PASK-2, J11 JST-EH Connector - S02B-PASK-2, J12 RGB LED HEADEER, J2 GROUND HEADER, J3 jumper, J4 jumper, J5 jumper, J6 jumper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

Commit message: update
Routing:
- net Board_0-GND: track 441.4 -> 471.4 mm
- net Board_0-Net-(HPTRS2-Pad3): track 166.9 -> 168.5 mm
- net Board_0-Net-(HPTRS2-Pad4): track 147.4 -> 146.8 mm
